Commit message: Migrated sections of blimp_description

File: src/blimp_description/urdf/blimp_base.xacro (robot description, xacro)
@@ -2,17 +2,17 @@
 <robot name="blimp" xmlns:xacro="http://ros.org/wiki/xacro">
 	<!--*****************  component description  *****************-->
-	<xacro:include filename="$(find-pkg-share blimp_description)/urdf/plugin_control.xacro" />
-	<xacro:include filename="$(find-pkg-share blimp_description)/urdf/plugin_sensors.xacro" />
-	<xacro:include filename="$(find-pkg-share blimp_description)/urdf/plugin_physics.xacro" />
+	<xacro:include filename="$(find blimp_description)/urdf/plugin_control.xacro" />
+	<xacro:include filename="$(find blimp_description)/urdf/plugin_sensors.xacro" />
+	<xacro:include filename="$(find blimp_description)/urdf/plugin_physics.xacro" />
 	<!--*****************  property description  *****************-->
-	<xacro:include filename="$(find-pkg-share blimp_description)/urdf/description_property.xacro"/>
+	<xacro:include filename="$(find blimp_description)/urdf/description_property.xacro"/>
 	<!--*****************  mechanics description	 *****************-->
-	<xacro:include filename="$(find-pkg-share blimp_description)/urdf/model_xacro.xacro" />
-	<xacro:include filename="$(find-pkg-share blimp_description)/urdf/description_link.xacro"/>
+	<xacro:include filename="$(find blimp_description)/urdf/model_xacro.xacro" />
+	<xacro:include filename="$(find blimp_description)/urdf/description_link.xacro"/>
 	<!--*****************  controller description  *****************-->
-	<xacro:include filename="$(find-pkg-share blimp_description)/urdf/description_controller.xacro"/>
+	<xacro:include filename="$(find blimp_description)/urdf/description_controller.xacro"/>
 	<!--*****************  sensor description  *****************-->
-	<xacro:include filename="$(find-pkg-share blimp_description)/urdf/description_sensor.xacro"/>
+	<xacro:include filename="$(find blimp_description)/urdf/description_sensor.xacro"/>
 	<!--*****************  physics and extra plugins description  *****************-->
-	<xacro:include filename="$(find-pkg-share blimp_description)/urdf/description_plugin.xacro"/>
+	<xacro:include filename="$(find blimp_description)/urdf/description_plugin.xacro"/>
 </robot>

File: src/blimp_description/urdf/description_controller.xacro (robot description, xacro)
@@ -1,8 +1,6 @@
 <?xml version="1.0" ?>
 <robot xmlns:xacro="http://ros.org/wiki/xacro">
-	<!-- ROS2 Control Interface -->
+	<!-- ROS2 Control Interface - Actually call it! -->
 	<xacro:ros2_control_interface namespace="${namespace}" />
-	<!-- Controller Plugin -->
-	<xacro:controller_plugin_macro namespace="${namespace}" imu_sub_topic="imu" />
 	<!-- Instantiate mavlink telemetry interface (placeholder for PX4 migration) -->
 	<xacro:if value="$(arg enable_mavlink_interface)">
@@ -59,4 +57,27 @@
 		actuator_name="motor1">
 	</xacro:transmission_macro>
-	<!-- Additional transmissions... -->
+	<xacro:transmission_macro
+		namespace="${namespace}"
+		joint_name="bot_rud_part1_bot_rud_joint_link_joint"
+		trans_name="tran2"
+		actuator_name="motor2">
+	</xacro:transmission_macro>
+	<xacro:transmission_macro
+		namespace="${namespace}"
+		joint_name="top_rud_part1_top_rud_joint_link_joint"
+		trans_name="tran3"
+		actuator_name="motor3">
+	</xacro:transmission_macro>
+	<xacro:transmission_macro
+		namespace="${namespace}"
+		joint_name="left_elv_part1_left_elv_joint_link_joint"
+		trans_name="tran4"
+		actuator_name="motor4">
+	</xacro:transmission_macro>
+	<xacro:transmission_macro
+		namespace="${namespace}"
+		joint_name="right_elv_part1_right_elv_joint_link_joint"
+		trans_name="tran5"
+		actuator_name="motor5">
+	</xacro:transmission_macro>
 </robot>

File: src/blimp_description/urdf/description_link.xacro (robot description, xacro)
@@ -464,3 +464,87 @@
       		<child link="right_elv_part2_link" />
     	</joint>
+<!-- IMU sensor link -->
+<link name="imu_link">
+	<inertial>
+		<mass value="0.015"/>
+		<origin xyz="0 0 0" rpy="0 0 0"/>
+		<inertia ixx="0.00001" ixy="0.0" ixz="0.0" iyy="0.00001" iyz="0.0" izz="0.00001"/>
+	</inertial>
+	<visual>
+		<origin xyz="0 0 0" rpy="0 0 0"/>
+		<geometry>
+			<box size="0.02 0.02 0.01"/>
+		</geometry>
+		<material name="imu_material">
+			<color rgba="0.1 0.1 0.8 1.0"/>
+		</material>
+	</visual>
+	<collision>
+		<origin xyz="0 0 0" rpy="0 0 0"/>
+		<geometry>
+			<box size="0.02 0.02 0.01"/>
+		</geometry>
+	</collision>
+</link>
+<joint name="blimp_body_imu_joint" type="fixed">
+	<origin xyz="0.0 0.0 0.0" rpy="0 0 0"/>
+	<parent link="blimp_body_link"/>
+	<child link="imu_link"/>
+</joint>
+<!-- GPS sensor link -->
+<link name="gps_link">
+	<inertial>
+		<mass value="0.015"/>
+		<origin xyz="0 0 0" rpy="0 0 0"/>
+		<inertia ixx="0.00001" ixy="0.0" ixz="0.0" iyy="0.00001" iyz="0.0" izz="0.00001"/>
+	</inertial>
+	<visual>
+		<origin xyz="0 0 0" rpy="0 0 0"/>
+		<geometry>
+			<cylinder radius="0.02" length="0.05"/>
+		</geometry>
+		<material name="gps_material">
+			<color rgba="0.8 0.8 0.1 1.0"/>
+		</material>
+	</visual>
+	<collision>
+		<origin xyz="0 0 0" rpy="0 0 0"/>
+		<geometry>
+			<cylinder radius="0.02" length="0.05"/>
+		</geometry>
+	</collision>
+</link>
+<joint name="blimp_body_gps_joint" type="fixed">
+	<origin xyz="0.0 0.0 0.1" rpy="0 0 0"/>
+	<parent link="blimp_body_link"/>
+	<child link="gps_link"/>
+</joint>
+<!-- Magnetometer sensor link -->
+<link name="magnetometer_link">
+	<inertial>
+		<mass value="0.010"/>
+		<origin xyz="0 0 0" rpy="0 0 0"/>
+		<inertia ixx="0.00001" ixy="0.0" ixz="0.0" iyy="0.00001" iyz="0.0" izz="0.00001"/>
+	</inertial>
+	<visual>
+		<origin xyz="0 0 0" rpy="0 0 0"/>
+		<geometry>
+			<box size="0.015 0.015 0.008"/>
+		</geometry>
+		<material name="mag_material">
+			<color rgba="0.8 0.1 0.1 1.0"/>
+		</material>
+	</visual>
+	<collision>
+		<origin xyz="0 0 0" rpy="0 0 0"/>
+		<geometry>
+			<box size="0.015 0.015 0.008"/>
+		</geometry>
+	</collision>
+</link>
+<joint name="blimp_body_magnetometer_joint" type="fixed">
+	<origin xyz="0.05 0.0 0.0" rpy="0 0 0"/>
+	<parent link="blimp_body_link"/>
+	<child link="magnetometer_link"/>
+</joint>
 </robot>

File: src/blimp_description/urdf/description_property.xacro (robot description, xacro)
@@ -17,4 +17,21 @@
 	<xacro:property name="mesh_file_blimp_rud_part2" value="package://blimp_description/meshes/blimp_fin/blimp_top_rud_part2_v5.dae" />
 	<xacro:property name="mesh_file_blimp_bot_rud_part1" value="package://blimp_description/meshes/blimp_fin/blimp_bot_rud_part1_v3.dae" />
+	<!-- Volume and gas properties -->
+	<xacro:property name="volume_total" value="${volume_blimp_body}" />
+	<xacro:property name="helium_mass" value="1.723" /> <!-- kg -->
+	<!-- Sensor noise parameters for Gazebo Harmonic -->
+	<xacro:property name="gyroscope_noise_density" value="0.0003394" />
+	<xacro:property name="gyroscope_random_walk" value="0.000038785" />
+	<xacro:property name="gyroscope_bias_correlation_time" value="1000.0" />
+	<xacro:property name="gyroscope_turn_on_bias_sigma" value="0.0087" />
+	<xacro:property name="accelerometer_noise_density" value="0.004" />
+	<xacro:property name="accelerometer_random_walk" value="0.006" />
+	<xacro:property name="accelerometer_bias_correlation_time" value="300.0" />
+	<xacro:property name="accelerometer_turn_on_bias_sigma" value="0.1960" />
+	<!-- Additional missing fin definitions -->
+	<xacro:property name="area_fin_total" value="${area_fin * 6}" /> <!-- 6 fins total -->
+	<xacro:property name="area_body_side" value="5.0" /> <!-- Side projection area -->
+	<!-- Gazebo Harmonic controller parameters -->
+	<xacro:property name="controller_update_rate" value="100" /> <!-- Hz -->
 	<!-- mass [kg] -->
 	<!-- Modified mass for convenience -->
@@ -86,5 +103,5 @@
 	<xacro:property name="area_body_front" value="3.14"/> <!-- [m^2] -->
 	<!-- inertia [kg m^2] [kg m^2] [kg m^2] [kg m^2] [kg m^2] [kg m^2] -->
-	<xacro:include filename="$(find-pkg-share blimp_description)/urdf/inertia_calculator.xacro"/>
+	<xacro:include filename="$(find blimp_description)/urdf/inertia_calculator.xacro"/>
 	<xacro:property name="inertia_blimp_body">
     		<xacro:hollow_cylinder_inertia r1="${radius_blimp_body - length_blimp_skin}" r2="${radius_blimp_body}" h="${length_blimp_body}" mass="${mass_blimp_body_without_gas}"/> <!--TODO: better use hollow ellipse-->

File: src/blimp_description/urdf/description_sensor.xacro (robot description, xacro)
@@ -29,5 +29,5 @@
 			<xacro:insert_block name="origin_camera" />
 		</xacro:vi_sensor_camera_macro>-->
-		<xacro:include filename="$(find-pkg-share blimp_description)/urdf/asus_camera.urdf.xacro" />
+		<xacro:include filename="$(find blimp_description)/urdf/asus_camera.urdf.xacro" />
 		<xacro:asus_camera
 		    name="xtion"

File: src/blimp_description/urdf/plugin_component_snippets.xacro (robot description, xacro)
@@ -1,5 +1,4 @@
 <?xml version="1.0"?>
 <robot xmlns:xacro="http://ros.org/wiki/xacro">
-  <xacro:property name="pi" value="3.14159265359" />
   <!-- =============================================================== -->
   <!-- ==================== LOGGING MACRO ========================== -->

File: src/blimp_description/urdf/plugin_control.xacro (robot description, xacro)
@@ -2,5 +2,5 @@
 <robot xmlns:xacro="http://ros.org/wiki/xacro">
   <!-- Include component snippets for macro definitions -->
-  <xacro:include filename="$(find-pkg-share blimp_description)/urdf/plugin_component_snippets.xacro" />
+  <xacro:include filename="$(find blimp_description)/urdf/plugin_component_snippets.xacro" />
   <!-- =============================================================== -->
   <!-- ==================== ROTOR MOTOR MACRO ====================== -->
@@ -12,7 +12,8 @@
       rolling_moment_coefficient">
     <!-- Gazebo Harmonic Multicopter Motor Model Plugin -->
-    <gazebo reference="${link_name}">
+    <gazebo>
       <plugin filename="gz-sim-multicopter-motor-model-system"
-              name="gz::sim::systems::MulticopterMotorModel">
+              name="motor_${motor_number}">
+        <robotNamespace>${robot_namespace}</robotNamespace>
         <jointName>${joint_name}</jointName>
         <linkName>${link_name}</linkName>
@@ -29,7 +30,4 @@
         <motorSpeedPubTopic>motor_speed/${motor_number}</motorSpeedPubTopic>
         <rotorVelocitySlowdownSim>1</rotorVelocitySlowdownSim>
-        <ros>
-          <namespace>${robot_namespace}</namespace>
-        </ros>
       </plugin>
     </gazebo>
@@ -60,6 +58,6 @@
       <joint name="base_stick_joint">
         <command_interface name="position">
-          <param name="min">-${100 * pi /180.0}</param>
-          <param name="max">${100 * pi /180.0}</param>
+          <param name="min">-1.745</param>
+          <param name="max">1.745</param>
         </command_interface>
         <state_interface name="position"/>
@@ -69,6 +67,6 @@
       <joint name="bot_rud_part1_bot_rud_joint_link_joint">
         <command_interface name="position">
-          <param name="min">-${60 * pi /180.0}</param>
-          <param name="max">${60 * pi /180.0}</param>
+          <param name="min">-1.047</param>
+          <param name="max">1.047</param>
         </command_interface>
         <state_interface name="position"/>
@@ -78,6 +76,6 @@
       <joint name="top_rud_part1_top_rud_joint_link_joint">
         <command_interface name="position">
-          <param name="min">-${60 * pi /180.0}</param>
-          <param name="max">${60 * pi /180.0}</param>
+          <param name="min">-1.047</param>
+          <param name="max">1.047</param>
         </command_interface>
         <state_interface name="position"/>
@@ -87,6 +85,6 @@
       <joint name="left_elv_part1_left_elv_joint_link_joint">
         <command_interface name="position">
-          <param name="min">-${60 * pi /180.0}</param>
-          <param name="max">${60 * pi /180.0}</param>
+          <param name="min">-1.047</param>
+          <param name="max">1.047</param>
         </command_interface>
         <state_interface name="position"/>
@@ -96,6 +94,6 @@
       <joint name="right_elv_part1_right_elv_joint_link_joint">
         <command_interface name="position">
-          <param name="min">-${60 * pi /180.0}</param>
-          <param name="max">${60 * pi /180.0}</param>
+          <param name="min">-1.047</param>
+          <param name="max">1.047</param>
         </command_interface>
         <state_interface name="position"/>
@@ -106,6 +104,6 @@
     <!-- Gazebo ROS2 Control Plugin -->
     <gazebo>
-      <plugin filename="gz_ros2_control-system" name="gz_ros2_control::GazeboSimROS2ControlPlugin">
-        <parameters>$(find-pkg-share blimp_description)/config/blimp_controllers.yaml</parameters>
+      <plugin filename="gz_ros2_control-system" name="gz_ros2_control::GzSimROS2ControlPlugin">
+        <parameters>$(find blimp_description)/config/controller_blimp.yaml</parameters>
         <ros>
           <namespace>${namespace}</namespace>
@@ -117,8 +115,6 @@
   <!-- ==================== MAVLINK INTERFACE (PLACEHOLDER) ======== -->
   <!-- =============================================================== -->
-  <!-- NOTE: This will need to be replaced with PX4/Pixhawk integration later -->
   <xacro:macro name="default_mavlink_interface" params="namespace imu_sub_topic rotor_count">
     <!-- Placeholder for future PX4 integration -->
-    <!-- For now, use ROS1_bridge for LibrePilot compatibility -->
     <gazebo>
       <plugin filename="gz-sim-joint-state-publisher-system"
@@ -135,5 +131,5 @@
   <!-- =============================================================== -->
   <xacro:macro name="controller_plugin_macro" params="namespace imu_sub_topic">
-    <!-- Custom ROS2 controller interface to replace rotors_simulator controller -->
+    <!-- Custom ROS2 controller interface -->
     <gazebo>
       <plugin filename="gz-sim-triggered-publisher-system" name="gz::sim::systems::TriggeredPublisher">

File: src/blimp_description/urdf/plugin_sensors.xacro (robot description, xacro)
@@ -2,5 +2,5 @@
 <robot xmlns:xacro="http://ros.org/wiki/xacro">
   <!-- Include component snippets for macro definitions -->
-  <xacro:include filename="$(find-pkg-share blimp_description)/urdf/plugin_component_snippets.xacro" />
+  <xacro:include filename="$(find blimp_description)/urdf/plugin_component_snippets.xacro" />
   <!-- =============================================================== -->
   <!-- ==================== IMU SENSOR MACRO ======================= -->

Commit message: Mesh migration

File: src/blimp_description/urdf/blimp_base.xacro (robot description, xacro)
@@ -1,4 +1,7 @@
 <?xml version="1.0" ?>
 <robot name="blimp" xmlns:xacro="http://ros.org/wiki/xacro">
+	<!-- Define M_PI for ROS2 xacro compatibility -->
+	<xacro:property name="M_PI" value="3.14159265359" />
+	<xacro:property name="PI" value="3.14159265359" />
 	<!--*****************  component description  *****************-->
 	<xacro:include filename="$(find blimp_description)/urdf/plugin_control.xacro" />
