Commit message: Debugging the launch progress

File: src/blimp_description/urdf/blimp_base.xacro (robot description, xacro)
@@ -5,4 +5,6 @@
   <xacro:property name="PI" value="3.14159265359" />
   <xacro:arg name="namespace" default="blimp"/>
+  <!-- ADDED: Missing launch argument that was referenced in launch files -->
+  <xacro:arg name="enable_custom_plugins" default="true"/>
   <!--*****************  component description  *****************-->
   <xacro:include filename="$(find blimp_description)/urdf/plugin_control.xacro" />
@@ -20,3 +22,7 @@
   <!--*****************  physics and extra plugins description  *****************-->
   <xacro:include filename="$(find blimp_description)/urdf/description_plugin.xacro"/>
+  <!-- ROS 2 Control hardware interface (Gazebo Harmonic) - FIXED -->
+  <gazebo>
+    <plugin name="gz_ros2_control" filename="gz_ros2_control-system"/>
+  </gazebo>
 </robot>

File: src/blimp_description/urdf/description_link.xacro (robot description, xacro)
@@ -190,6 +190,7 @@
   <link name="forward_lift_joint_link">
     <inertial>
-      <mass value="1e-3"/> <!-- MUST be non zero or link will be pruned -->
-      <inertia ixx="0.0" ixy="0.0" ixz="0.0" iyy="0.0" iyz="0.0" izz="0.0" />
+      <mass value="1e-3"/> <!-- Original ROS1 mass -->
+      <!-- FIXED: Minimal valid inertia for existing mass (ROS1 had zero - invalid in Gazebo Harmonic) -->
+      <inertia ixx="1e-6" ixy="0.0" ixz="0.0" iyy="1e-6" iyz="0.0" izz="1e-6" />
     </inertial>
     <visual>
@@ -207,6 +208,7 @@
   <link name="aft_lift_joint_link">
     <inertial>
-      <mass value="1e-3"/>
-      <inertia ixx="0.0" ixy="0.0" ixz="0.0" iyy="0.0" iyz="0.0" izz="0.0" />
+      <mass value="1e-3"/> <!-- Original ROS1 mass -->
+      <!-- FIXED: Minimal valid inertia for existing mass (ROS1 had zero - invalid in Gazebo Harmonic) -->
+      <inertia ixx="1e-6" ixy="0.0" ixz="0.0" iyy="1e-6" iyz="0.0" izz="1e-6" />
     </inertial>
     <visual>
@@ -248,4 +250,10 @@
       </joint>
   <link name="top_rud_joint_link">
+    <!-- ADDED: Minimal inertial properties required by Gazebo Harmonic (ROS1 had none) -->
+    <inertial>
+      <mass value="1e-6"/>
+      <origin xyz="0 0 0" rpy="0 0 0"/>
+      <inertia ixx="1e-9" ixy="0.0" ixz="0.0" iyy="1e-9" iyz="0.0" izz="1e-9" />
+    </inertial>
     <visual>
       <geometry>
@@ -304,4 +312,10 @@
       </joint>
   <link name="bot_rud_joint_link">
+    <!-- ADDED: Minimal inertial properties required by Gazebo Harmonic (ROS1 had none) -->
+    <inertial>
+      <mass value="1e-6"/>
+      <origin xyz="0 0 0" rpy="0 0 0"/>
+      <inertia ixx="1e-9" ixy="0.0" ixz="0.0" iyy="1e-9" iyz="0.0" izz="1e-9" />
+    </inertial>
     <visual>
       <geometry>
@@ -378,4 +392,10 @@
       </joint>
   <link name="left_elv_joint_link">
+    <!-- ADDED: Minimal inertial properties required by Gazebo Harmonic (ROS1 had none) -->
+    <inertial>
+      <mass value="1e-6"/>
+      <origin xyz="0 0 0" rpy="0 0 0"/>
+      <inertia ixx="1e-9" ixy="0.0" ixz="0.0" iyy="1e-9" iyz="0.0" izz="1e-9" />
+    </inertial>
     <visual>
       <geometry>
@@ -434,4 +454,10 @@
       </joint>
   <link name="right_elv_joint_link">
+    <!-- ADDED: Minimal inertial properties required by Gazebo Harmonic (ROS1 had none) -->
+    <inertial>
+      <mass value="1e-6"/>
+      <origin xyz="0 0 0" rpy="0 0 0"/>
+      <inertia ixx="1e-9" ixy="0.0" ixz="0.0" iyy="1e-9" iyz="0.0" izz="1e-9" />
+    </inertial>
     <visual>
       <geometry>
@@ -464,87 +490,13 @@
           <child link="right_elv_part2_link" />
       </joint>
-<!-- IMU sensor link -->
-<link name="imu_link">
-  <inertial>
-    <mass value="0.015"/>
-    <origin xyz="0 0 0" rpy="0 0 0"/>
-    <inertia ixx="0.00001" ixy="0.0" ixz="0.0" iyy="0.00001" iyz="0.0" izz="0.00001"/>
-  </inertial>
-  <visual>
-    <origin xyz="0 0 0" rpy="0 0 0"/>
-    <geometry>
-      <box size="0.02 0.02 0.01"/>
-    </geometry>
-    <material name="imu_material">
-      <color rgba="0.1 0.1 0.8 1.0"/>
-    </material>
-  </visual>
-  <collision>
-    <origin xyz="0 0 0" rpy="0 0 0"/>
-    <geometry>
-      <box size="0.02 0.02 0.01"/>
-    </geometry>
-  </collision>
-</link>
-<joint name="blimp_body_imu_joint" type="fixed">
-  <origin xyz="0.0 0.0 0.0" rpy="0 0 0"/>
-  <parent link="blimp_body_link"/>
-  <child link="imu_link"/>
-</joint>
-<!-- GPS sensor link -->
-<link name="gps_link">
-  <inertial>
-    <mass value="0.015"/>
-    <origin xyz="0 0 0" rpy="0 0 0"/>
-    <inertia ixx="0.00001" ixy="0.0" ixz="0.0" iyy="0.00001" iyz="0.0" izz="0.00001"/>
-  </inertial>
-  <visual>
-    <origin xyz="0 0 0" rpy="0 0 0"/>
-    <geometry>
-      <cylinder radius="0.02" length="0.05"/>
-    </geometry>
-    <material name="gps_material">
-      <color rgba="0.8 0.8 0.1 1.0"/>
-    </material>
-  </visual>
-  <collision>
-    <origin xyz="0 0 0" rpy="0 0 0"/>
-    <geometry>
-      <cylinder radius="0.02" length="0.05"/>
-    </geometry>
-  </collision>
-</link>
-<joint name="blimp_body_gps_joint" type="fixed">
-  <origin xyz="0.0 0.0 0.1" rpy="0 0 0"/>
-  <parent link="blimp_body_link"/>
-  <child link="gps_link"/>
-</joint>
-<!-- Magnetometer sensor link -->
-<link name="magnetometer_link">
-  <inertial>
-    <mass value="0.010"/>
-    <origin xyz="0 0 0" rpy="0 0 0"/>
-    <inertia ixx="0.00001" ixy="0.0" ixz="0.0" iyy="0.00001" iyz="0.0" izz="0.00001"/>
-  </inertial>
-  <visual>
-    <origin xyz="0 0 0" rpy="0 0 0"/>
-    <geometry>
-      <box size="0.015 0.015 0.008"/>
-    </geometry>
-    <material name="mag_material">
-      <color rgba="0.8 0.1 0.1 1.0"/>
-    </material>
-  </visual>
-  <collision>
-    <origin xyz="0 0 0" rpy="0 0 0"/>
-    <geometry>
-      <box size="0.015 0.015 0.008"/>
-    </geometry>
-  </collision>
-</link>
-<joint name="blimp_body_magnetometer_joint" type="fixed">
-  <origin xyz="0.05 0.0 0.0" rpy="0 0 0"/>
-  <parent link="blimp_body_link"/>
-  <child link="magnetometer_link"/>
-</joint>
+<!-- REMOVED: Hardcoded sensor links - these are now handled by sensor plugin macros -->
+<!-- The following hardcoded sensor links were causing duplicates:
+     - imu_link (handled by IMU plugin)
+     - gps_link (handled by GPS plugin)
+     - magnetometer_link (handled by magnetometer plugin)
+     These are properly created by the sensor plugin system in:
+     - description_sensor.xacro
+     - plugin_sensors.xacro
+     - plugin_component_snippets.xacro
+-->
 </robot>

File: src/blimp_description/urdf/description_plugin.xacro (robot description, xacro)
@@ -4,5 +4,6 @@
   <xacro:if value="$(arg enable_wind)">
     <gazebo>
-      <plugin filename="libnormwind_plugin.so" name="normwind_plugin::NormWindPlugin">
+      <!-- FIXED: Correct Gazebo Harmonic plugin filename format -->
+      <plugin filename="normwind_plugin" name="normwind_plugin::NormWindPlugin">
         <robotNamespace>${namespace}</robotNamespace>
         <linkName>blimp_body_link</linkName>
@@ -22,5 +23,6 @@
     <!-- Main body aerodynamics -->
     <gazebo>
-      <plugin name="blimp_body_finliftdrag" filename="libfinliftdrag_plugin.so">
+      <!-- FIXED: Correct Gazebo Harmonic plugin filename format -->
+      <plugin name="blimp_body_finliftdrag" filename="finliftdrag_plugin">
         <robotNamespace>${namespace}</robotNamespace>
         <link_name>blimp_body_link</link_name>
@@ -44,5 +46,6 @@
     <!-- Bottom rudder aerodynamics -->
     <gazebo>
-      <plugin name="bot_rud_finliftdrag" filename="libfinliftdrag_plugin.so">
+      <!-- FIXED: Correct Gazebo Harmonic plugin filename format -->
+      <plugin name="bot_rud_finliftdrag" filename="finliftdrag_plugin">
         <robotNamespace>${namespace}</robotNamespace>
         <link_name>bot_rud_part1_link</link_name>
@@ -68,5 +71,6 @@
     <!-- Top rudder aerodynamics -->
     <gazebo>
-      <plugin name="top_rud_finliftdrag" filename="libfinliftdrag_plugin.so">
+      <!-- FIXED: Correct Gazebo Harmonic plugin filename format -->
+      <plugin name="top_rud_finliftdrag" filename="finliftdrag_plugin">
         <robotNamespace>${namespace}</robotNamespace>
         <link_name>top_rud_part1_link</link_name>
@@ -89,5 +93,6 @@
   <!-- Buoyancy Plugin - Using your migrated dynamicvolume_plugin -->
   <gazebo>
-    <plugin name="dynamicvolume_plugin" filename="libdynamicvolume_plugin.so">
+    <!-- FIXED: Correct Gazebo Harmonic plugin filename format -->
+    <plugin name="dynamicvolume_plugin" filename="dynamicvolume_plugin">
       <robotNamespace>${namespace}</robotNamespace>
       <linkName>blimp_body_link</linkName>
@@ -105,8 +110,10 @@
     </plugin>
   </gazebo>
-  <!-- MOTOR PLUGINS - FIXED syntax for Gazebo Harmonic -->
+  <!-- MOTOR PLUGINS  -->
   <!-- Left blade motor -->
   <gazebo>
-    <plugin filename="gz-sim-multicopter-motor-model-system" name="gz::sim::systems::MulticopterMotorModel">
+    <!-- FIXED: Correct Gazebo Harmonic built-in plugin filename -->
+    <plugin filename="gz-sim-multicopter-motor-model-system"
+            name="gz::sim::systems::MulticopterMotorModel">
       <robotNamespace>${namespace}</robotNamespace>
       <linkName>left_blade_link</linkName>
@@ -119,16 +126,19 @@
       <momentConstant>0.016</momentConstant>
       <commandSubTopic>command/motor_speed</commandSubTopic>
-      <!-- FIXED: Use actuator_number instead of motorNumber -->
       <actuator_number>0</actuator_number>
       <rotorDragCoefficient>8.06428e-05</rotorDragCoefficient>
       <rollingMomentCoefficient>1e-06</rollingMomentCoefficient>
       <motorSpeedPubTopic>motor_speed/0</motorSpeedPubTopic>
-      <!-- ADDED: Missing motor type specification -->
       <motorType>velocity</motorType>
+      <ros>
+        <namespace>${namespace}</namespace>
+      </ros>
     </plugin>
   </gazebo>
   <!-- Right blade motor -->
   <gazebo>
-    <plugin filename="gz-sim-multicopter-motor-model-system" name="gz::sim::systems::MulticopterMotorModel">
+    <!-- FIXED: Correct Gazebo Harmonic built-in plugin filename -->
+    <plugin filename="gz-sim-multicopter-motor-model-system"
+            name="gz::sim::systems::MulticopterMotorModel">
       <robotNamespace>${namespace}</robotNamespace>
       <linkName>right_blade_link</linkName>
@@ -141,16 +151,19 @@
       <momentConstant>0.016</momentConstant>
       <commandSubTopic>command/motor_speed</commandSubTopic>
-      <!-- FIXED: Use actuator_number instead of motorNumber -->
       <actuator_number>1</actuator_number>
       <rotorDragCoefficient>8.06428e-05</rotorDragCoefficient>
       <rollingMomentCoefficient>1e-06</rollingMomentCoefficient>
       <motorSpeedPubTopic>motor_speed/1</motorSpeedPubTopic>
-      <!-- ADDED: Missing motor type specification -->
       <motorType>velocity</motorType>
+      <ros>
+        <namespace>${namespace}</namespace>
+      </ros>
     </plugin>
   </gazebo>
   <!-- Bottom rudder motor -->
   <gazebo>
-    <plugin filename="gz-sim-multicopter-motor-model-system" name="gz::sim::systems::MulticopterMotorModel">
+    <!-- FIXED: Correct Gazebo Harmonic built-in plugin filename -->
+    <plugin filename="gz-sim-multicopter-motor-model-system"
+            name="gz::sim::systems::MulticopterMotorModel">
       <robotNamespace>${namespace}</robotNamespace>
       <linkName>bot_rud_motor_link</linkName>
@@ -163,75 +176,31 @@
       <momentConstant>0.016</momentConstant>
       <commandSubTopic>command/motor_speed</commandSubTopic>
-      <!-- FIXED: Use actuator_number instead of motorNumber -->
       <actuator_number>2</actuator_number>
       <rotorDragCoefficient>8.06428e-05</rotorDragCoefficient>
       <rollingMomentCoefficient>1e-06</rollingMomentCoefficient>
       <motorSpeedPubTopic>motor_speed/2</motorSpeedPubTopic>
-      <!-- ADDED: Missing motor type specification -->
       <motorType>velocity</motorType>
-    </plugin>
-  </gazebo>
-  <!-- SENSOR PLUGINS - Using Gazebo Harmonic built-ins -->
-  <!-- IMU sensor -->
-  <xacro:if value="$(arg enable_sensors)">
-    <gazebo reference="imu_link">
-      <sensor type="imu" name="blimp_imu">
-        <pose>0 0 0 0 0 0</pose>
-        <topic>${namespace}/imu</topic>
-        <update_rate>1000</update_rate>
-        <imu>
-          <angular_velocity>
-            <x>
-              <noise type="gaussian">
-                <mean>0.0</mean>
-                <stddev>0.0003394</stddev>
-              </noise>
-            </x>
-            <y>
-              <noise type="gaussian">
-                <mean>0.0</mean>
-                <stddev>0.0003394</stddev>
-              </noise>
-            </y>
-            <z>
-              <noise type="gaussian">
-                <mean>0.0</mean>
-                <stddev>0.0003394</stddev>
-              </noise>
-            </z>
-          </angular_velocity>
-          <linear_acceleration>
-            <x>
-              <noise type="gaussian">
-                <mean>0.0</mean>
-                <stddev>0.004</stddev>
-              </noise>
-            </x>
-            <y>
-              <noise type="gaussian">
-                <mean>0.0</mean>
-                <stddev>0.004</stddev>
-              </noise>
-            </y>
-            <z>
-              <noise type="gaussian">
-                <mean>0.0</mean>
-                <stddev>0.004</stddev>
-              </noise>
-            </z>
-          </linear_acceleration>
-        </imu>
-        <plugin filename="gz-sim-imu-system" name="gz::sim::systems::Imu">
-          <ros>
-            <namespace>${namespace}</namespace>
-          </ros>
-        </plugin>
-      </sensor>
-    </gazebo>
-  </xacro:if>
-  <!-- Ground Truth Odometry -->
+      <ros>
+        <namespace>${namespace}</namespace>
+      </ros>
+    </plugin>
+  </gazebo>
+  <!-- REMOVED: Hardcoded sensor plugins that referenced deleted links -->
+  <!-- The following sensor plugins were removed because they referenced
+       hardcoded links (imu_link, gps_link, magnetometer_link) that we deleted:
+       - IMU sensor plugin (now handled by sensor plugin macros in description_sensor.xacro)
+       - GPS sensor plugin (now handled by sensor plugin macros in description_sensor.xacro)
+       - Magnetometer sensor plugin (can be added via sensor macros if needed)
+       These sensors are properly created by the sensor plugin system in:
+       - description_sensor.xacro calls the sensor macros
+       - plugin_sensors.xacro defines the sensor macros
+       - The macros create both the links AND the sensor plugins
+  -->
+  <!-- Ground Truth Odometry - This doesn't reference a specific sensor link -->
   <xacro:if value="$(arg enable_ground_truth)">
     <gazebo>
-      <plugin filename="gz-sim-odometry-publisher-system" name="gz::sim::systems::OdometryPublisher">
+      <!-- FIXED: Correct Gazebo Harmonic built-in plugin filename -->
+      <plugin filename="gz-sim-odometry-publisher-system"
+              name="gz::sim::systems::OdometryPublisher">
         <ros>
           <namespace>${namespace}</namespace>

File: src/blimp_description/urdf/model_xacro.xacro (robot description, xacro)
@@ -140,28 +140,35 @@
   <!-- =============================================================== -->
   <!-- Spring/flexible joint macro for realistic deformation -->
+  <!-- FIXED: Using original ROS1 inertia values -->
   <xacro:macro name="spring"
     params="robot_namespace link_name parent strength_factor:=1.0
-            roll_factor:=1.0 pitch_factor:=1.0 yaw_factor:=1.0 *origin">
+            roll_factor:=1.0 pitch_factor:=5.0 yaw_factor:=10.0 *origin">
     <!-- Create intermediate links for 3-DOF flexibility -->
+    <!-- FIXED: Original ROS1 values -->
     <link name="${link_name}_link0">
       <inertial>
-        <mass value="1e-6"/>
+        <mass value="0.0001"/><!-- MUST be non zero or the link will be pruned by gazebo -->
         <origin xyz="0 0 0" rpy="0 0 0"/>
-        <inertia ixx="1e-9" ixy="0" ixz="0" iyy="1e-9" iyz="0" izz="1e-9"/>
+        <inertia ixx="0.01" ixy="0.0" ixz="0.0" iyy="0.01" iyz="0.0" izz="0.01" />
       </inertial>
     </link>
     <link name="${link_name}_link1">
       <inertial>
-        <mass value="1e-6"/>
+        <mass value="0.0001"/><!-- MUST be non zero or the link will be pruned by gazebo -->
         <origin xyz="0 0 0" rpy="0 0 0"/>
-        <inertia ixx="1e-9" ixy="0" ixz="0" iyy="1e-9" iyz="0" izz="1e-9"/>
-      </inertial>
-    </link>
-    <link name="${link_name}_link">
-      <inertial>
-        <mass value="1e-6"/>
+        <inertia ixx="0.01" ixy="0.0" ixz="0.0" iyy="0.01" iyz="0.0" izz="0.01" />
+      </inertial>
+    </link>
+    <link name="${link_name}_link">
+      <inertial>
+        <mass value="0.0001"/><!-- MUST be non zero or the link will be pruned by gazebo -->
         <origin xyz="0 0 0" rpy="0 0 0"/>
-        <inertia ixx="1e-9" ixy="0" ixz="0" iyy="1e-9" iyz="0" izz="1e-9"/>
-      </inertial>
+        <inertia ixx="0.01" ixy="0.0" ixz="0.0" iyy="0.01" iyz="0.0" izz="0.01" />
+      </inertial>
+      <visual>
+        <geometry>
+          <cylinder radius="0.01" length="0.3"/>
+        </geometry>
+      </visual>
     </link>
     <!-- Joint chain for 3-DOF spring behavior -->

File: src/blimp_description/urdf/plugin_control.xacro (robot description, xacro)
@@ -33,4 +33,8 @@
         <!-- ADDED: Specify motor type to eliminate warning -->
         <motorType>velocity</motorType>
+        <!-- ADDED: ROS namespace configuration -->
+        <ros>
+          <namespace>${robot_namespace}</namespace>
+        </ros>
       </plugin>
     </gazebo>
@@ -105,7 +109,8 @@
       </joint>
     </ros2_control>
-    <!-- Gazebo ROS2 Control Plugin - FIXED PLUGIN NAME -->
+    <!-- Gazebo ROS2 Control Plugin - FIXED -->
     <gazebo>
-      <plugin filename="gz_ros2_control-system" name="gz_ros2_control::GazeboSimROS2ControlPlugin">
+      <plugin filename="gz_ros2_control-system"
+              name="gz_ros2_control::GazeboSimROS2ControlPlugin">
         <parameters>$(find blimp_description)/resource/controller_blimp.yaml</parameters>
         <ros>
@@ -136,5 +141,6 @@
     <!-- Custom ROS2 controller interface -->
     <gazebo>
-      <plugin filename="gz-sim-triggered-publisher-system" name="gz::sim::systems::TriggeredPublisher">
+      <plugin filename="gz-sim-triggered-publisher-system"
+              name="gz::sim::systems::TriggeredPublisher">
         <input type="gz.msgs.Twist" topic="/${namespace}/cmd_vel">
           <match field="linear.x">0.0</match>
