Commit message: Fully debugged launch -meshes

File: src/blimp_description/urdf/blimp_base.xacro (robot description, xacro)
@@ -5,6 +5,17 @@
   <xacro:property name="PI" value="3.14159265359" />
   <xacro:arg name="namespace" default="blimp"/>
-  <!-- ADDED: Missing launch argument that was referenced in launch files -->
+  <xacro:arg name="uav_name" default="blimp"/>
+  <!-- FIXED: Added all missing launch arguments that are referenced in included files -->
   <xacro:arg name="enable_custom_plugins" default="true"/>
+  <xacro:arg name="enable_meshes" default="true"/>
+  <xacro:arg name="enable_wind" default="false"/>
+  <xacro:arg name="enable_physics" default="true"/>
+  <xacro:arg name="enable_sensors" default="true"/>
+  <xacro:arg name="enable_logging" default="false"/>
+  <xacro:arg name="enable_ground_truth" default="true"/>
+  <xacro:arg name="enable_mavlink_interface" default="false"/>
+  <xacro:arg name="log_file" default="blimp"/>
+  <xacro:arg name="wait_to_record_bag" default="false"/>
+  <xacro:arg name="is_input_joystick" default="false"/>
   <!--*****************  component description  *****************-->
   <xacro:include filename="$(find blimp_description)/urdf/plugin_control.xacro" />
@@ -22,7 +33,12 @@
   <!--*****************  physics and extra plugins description  *****************-->
   <xacro:include filename="$(find blimp_description)/urdf/description_plugin.xacro"/>
-  <!-- ROS 2 Control hardware interface (Gazebo Harmonic) - FIXED -->
+  <!-- ROS 2 Control hardware interface (Gazebo Harmonic) -->
   <gazebo>
-    <plugin name="gz_ros2_control" filename="gz_ros2_control-system"/>
+    <plugin name="gz_ros2_control::GazeboSimROS2ControlPlugin" filename="gz_ros2_control-system">
+      <parameters>$(find blimp_description)/resource/controller_blimp.yaml</parameters>
+      <ros>
+        <namespace>$(arg namespace)</namespace>
+      </ros>
+    </plugin>
   </gazebo>
 </robot>

File: src/blimp_description/urdf/description_plugin.xacro (robot description, xacro)
@@ -92,109 +92,102 @@
   </xacro:if>
   <!-- Buoyancy Plugin - Using your migrated dynamicvolume_plugin -->
-  <gazebo>
-    <!-- FIXED: Correct Gazebo Harmonic plugin filename format -->
-    <plugin name="dynamicvolume_plugin" filename="dynamicvolume_plugin">
-      <robotNamespace>${namespace}</robotNamespace>
-      <linkName>blimp_body_link</linkName>
-      <dynamicVolumeTopic>dynamic_volume</dynamicVolumeTopic>
-      <heliumMassTopic>helium_mass</heliumMassTopic>
-      <heliumMassKG>1.0</heliumMassKG>
-      <refAlt>0</refAlt>
-      <fluidDensity>1.2041</fluidDensity>
-      <frameId>world</frameId>
-      <!-- Link volume properties -->
-      <link name="blimp_body_link">
-        <volume>10.472</volume>
-        <center_of_volume>0 0 0</center_of_volume>
-      </link>
-    </plugin>
-  </gazebo>
-  <!-- MOTOR PLUGINS  -->
-  <!-- Left blade motor -->
-  <gazebo>
-    <!-- FIXED: Correct Gazebo Harmonic built-in plugin filename -->
-    <plugin filename="gz-sim-multicopter-motor-model-system"
-            name="gz::sim::systems::MulticopterMotorModel">
-      <robotNamespace>${namespace}</robotNamespace>
-      <linkName>left_blade_link</linkName>
-      <jointName>stick_left_blade_joint</jointName>
-      <turningDirection>ccw</turningDirection>
-      <timeConstantUp>0.0125</timeConstantUp>
-      <timeConstantDown>0.025</timeConstantDown>
-      <maxRotVelocity>838</maxRotVelocity>
-      <motorConstant>8.54858e-06</motorConstant>
-      <momentConstant>0.016</momentConstant>
-      <commandSubTopic>command/motor_speed</commandSubTopic>
-      <actuator_number>0</actuator_number>
-      <rotorDragCoefficient>8.06428e-05</rotorDragCoefficient>
-      <rollingMomentCoefficient>1e-06</rollingMomentCoefficient>
-      <motorSpeedPubTopic>motor_speed/0</motorSpeedPubTopic>
-      <motorType>velocity</motorType>
-      <ros>
-        <namespace>${namespace}</namespace>
-      </ros>
-    </plugin>
-  </gazebo>
-  <!-- Right blade motor -->
-  <gazebo>
-    <!-- FIXED: Correct Gazebo Harmonic built-in plugin filename -->
-    <plugin filename="gz-sim-multicopter-motor-model-system"
-            name="gz::sim::systems::MulticopterMotorModel">
-      <robotNamespace>${namespace}</robotNamespace>
-      <linkName>right_blade_link</linkName>
-      <jointName>stick_right_blade_joint</jointName>
-      <turningDirection>cw</turningDirection>
-      <timeConstantUp>0.0125</timeConstantUp>
-      <timeConstantDown>0.025</timeConstantDown>
-      <maxRotVelocity>838</maxRotVelocity>
-      <motorConstant>8.54858e-06</motorConstant>
-      <momentConstant>0.016</momentConstant>
-      <commandSubTopic>command/motor_speed</commandSubTopic>
-      <actuator_number>1</actuator_number>
-      <rotorDragCoefficient>8.06428e-05</rotorDragCoefficient>
-      <rollingMomentCoefficient>1e-06</rollingMomentCoefficient>
-      <motorSpeedPubTopic>motor_speed/1</motorSpeedPubTopic>
-      <motorType>velocity</motorType>
-      <ros>
-        <namespace>${namespace}</namespace>
-      </ros>
-    </plugin>
-  </gazebo>
-  <!-- Bottom rudder motor -->
-  <gazebo>
-    <!-- FIXED: Correct Gazebo Harmonic built-in plugin filename -->
-    <plugin filename="gz-sim-multicopter-motor-model-system"
-            name="gz::sim::systems::MulticopterMotorModel">
-      <robotNamespace>${namespace}</robotNamespace>
-      <linkName>bot_rud_motor_link</linkName>
-      <jointName>bot_rud_part1_bot_rud_motor_joint</jointName>
-      <turningDirection>cw</turningDirection>
-      <timeConstantUp>0.0125</timeConstantUp>
-      <timeConstantDown>0.025</timeConstantDown>
-      <maxRotVelocity>838</maxRotVelocity>
-      <motorConstant>8.54858e-06</motorConstant>
-      <momentConstant>0.016</momentConstant>
-      <commandSubTopic>command/motor_speed</commandSubTopic>
-      <actuator_number>2</actuator_number>
-      <rotorDragCoefficient>8.06428e-05</rotorDragCoefficient>
-      <rollingMomentCoefficient>1e-06</rollingMomentCoefficient>
-      <motorSpeedPubTopic>motor_speed/2</motorSpeedPubTopic>
-      <motorType>velocity</motorType>
-      <ros>
-        <namespace>${namespace}</namespace>
-      </ros>
-    </plugin>
-  </gazebo>
-  <!-- REMOVED: Hardcoded sensor plugins that referenced deleted links -->
-  <!-- The following sensor plugins were removed because they referenced
-       hardcoded links (imu_link, gps_link, magnetometer_link) that we deleted:
-       - IMU sensor plugin (now handled by sensor plugin macros in description_sensor.xacro)
-       - GPS sensor plugin (now handled by sensor plugin macros in description_sensor.xacro)
-       - Magnetometer sensor plugin (can be added via sensor macros if needed)
-       These sensors are properly created by the sensor plugin system in:
-       - description_sensor.xacro calls the sensor macros
-       - plugin_sensors.xacro defines the sensor macros
-       - The macros create both the links AND the sensor plugins
-  -->
+  <xacro:if value="$(arg enable_custom_plugins)">
+    <gazebo>
+      <!-- FIXED: Correct Gazebo Harmonic plugin filename format -->
+      <plugin name="dynamicvolume_plugin" filename="dynamicvolume_plugin">
+        <robotNamespace>${namespace}</robotNamespace>
+        <linkName>blimp_body_link</linkName>
+        <dynamicVolumeTopic>dynamic_volume</dynamicVolumeTopic>
+        <heliumMassTopic>helium_mass</heliumMassTopic>
+        <heliumMassKG>1.0</heliumMassKG>
+        <refAlt>0</refAlt>
+        <fluidDensity>1.2041</fluidDensity>
+        <frameId>world</frameId>
+        <!-- Link volume properties -->
+        <link name="blimp_body_link">
+          <volume>10.472</volume>
+          <center_of_volume>0 0 0</center_of_volume>
+        </link>
+      </plugin>
+    </gazebo>
+  </xacro:if>
+  <!-- MOTOR PLUGINS - FIXED: Conditional inclusion -->
+  <xacro:if value="$(arg enable_physics)">
+    <!-- Left blade motor -->
+    <gazebo>
+      <!-- FIXED: Correct Gazebo Harmonic built-in plugin filename -->
+      <plugin filename="gz-sim-multicopter-motor-model-system"
+              name="gz::sim::systems::MulticopterMotorModel">
+        <robotNamespace>${namespace}</robotNamespace>
+        <linkName>left_blade_link</linkName>
+        <jointName>stick_left_blade_joint</jointName>
+        <turningDirection>ccw</turningDirection>
+        <timeConstantUp>0.0125</timeConstantUp>
+        <timeConstantDown>0.025</timeConstantDown>
+        <maxRotVelocity>838</maxRotVelocity>
+        <motorConstant>8.54858e-06</motorConstant>
+        <momentConstant>0.016</momentConstant>
+        <commandSubTopic>command/motor_speed</commandSubTopic>
+        <actuator_number>0</actuator_number>
+        <rotorDragCoefficient>8.06428e-05</rotorDragCoefficient>
+        <rollingMomentCoefficient>1e-06</rollingMomentCoefficient>
+        <motorSpeedPubTopic>motor_speed/0</motorSpeedPubTopic>
+        <motorType>velocity</motorType>
+        <ros>
+          <namespace>${namespace}</namespace>
+        </ros>
+      </plugin>
+    </gazebo>
+    <!-- Right blade motor -->
+    <gazebo>
+      <!-- FIXED: Correct Gazebo Harmonic built-in plugin filename -->
+      <plugin filename="gz-sim-multicopter-motor-model-system"
+              name="gz::sim::systems::MulticopterMotorModel">
+        <robotNamespace>${namespace}</robotNamespace>
+        <linkName>right_blade_link</linkName>
+        <jointName>stick_right_blade_joint</jointName>
+        <turningDirection>cw</turningDirection>
+        <timeConstantUp>0.0125</timeConstantUp>
+        <timeConstantDown>0.025</timeConstantDown>
+        <maxRotVelocity>838</maxRotVelocity>
+        <motorConstant>8.54858e-06</motorConstant>
+        <momentConstant>0.016</momentConstant>
+        <commandSubTopic>command/motor_speed</commandSubTopic>
+        <actuator_number>1</actuator_number>
+        <rotorDragCoefficient>8.06428e-05</rotorDragCoefficient>
+        <rollingMomentCoefficient>1e-06</rollingMomentCoefficient>
+        <motorSpeedPubTopic>motor_speed/1</motorSpeedPubTopic>
+        <motorType>velocity</motorType>
+        <ros>
+          <namespace>${namespace}</namespace>
+        </ros>
+      </plugin>
+    </gazebo>
+    <!-- Bottom rudder motor -->
+    <gazebo>
+      <!-- FIXED: Correct Gazebo Harmonic built-in plugin filename -->
+      <plugin filename="gz-sim-multicopter-motor-model-system"
+              name="gz::sim::systems::MulticopterMotorModel">
+        <robotNamespace>${namespace}</robotNamespace>
+        <linkName>bot_rud_motor_link</linkName>
+        <jointName>bot_rud_part1_bot_rud_motor_joint</jointName>
+        <turningDirection>cw</turningDirection>
+        <timeConstantUp>0.0125</timeConstantUp>
+        <timeConstantDown>0.025</timeConstantDown>
+        <maxRotVelocity>838</maxRotVelocity>
+        <motorConstant>8.54858e-06</motorConstant>
+        <momentConstant>0.016</momentConstant>
+        <commandSubTopic>command/motor_speed</commandSubTopic>
+        <actuator_number>2</actuator_number>
+        <rotorDragCoefficient>8.06428e-05</rotorDragCoefficient>
+        <rollingMomentCoefficient>1e-06</rollingMomentCoefficient>
+        <motorSpeedPubTopic>motor_speed/2</motorSpeedPubTopic>
+        <motorType>velocity</motorType>
+        <ros>
+          <namespace>${namespace}</namespace>
+        </ros>
+      </plugin>
+    </gazebo>
+  </xacro:if>
   <!-- Ground Truth Odometry - This doesn't reference a specific sensor link -->
   <xacro:if value="$(arg enable_ground_truth)">

File: src/blimp_description/urdf/description_property.xacro (robot description, xacro)
@@ -4,17 +4,17 @@
   <xacro:property name="namespace" value="$(arg uav_name)" />
   <xacro:property name="air_density" value="1.2041"/> <!--[kg/m^3] Temperature 20celsius: 1.2041-->
-  <!-- meshes -->
+  <!-- meshes - FIXED: Use file:// paths for Gazebo Harmonic compatibility -->
   <xacro:property name="use_mesh_file" value="$(arg enable_meshes)" />
-    <xacro:property name="mesh_file_blimp_body" value="package://blimp_description/meshes/blimp_body/blimp_body_v4.dae" />
-  <xacro:property name="mesh_file_blimp_support" value="package://blimp_description/meshes/blimp_support/blimp_support_v5.dae" />
-  <xacro:property name="mesh_file_blimp_gondola" value="package://blimp_description/meshes/blimp_gondola/blimp_gondola_v4.dae" />
-  <xacro:property name="mesh_file_blimp_wing" value="package://blimp_description/meshes/blimp_wing/blimp_wing_v2.dae" />
-  <xacro:property name="mesh_file_blimp_stick" value="package://blimp_description/meshes/blimp_wing/blimp_stick_v2.dae" />
-  <xacro:property name="mesh_file_propeller_cw" value="package://blimp_description/meshes/blimp_propeller/blimp_right_propeller_cw_v3.dae" />
-  <xacro:property name="mesh_file_propeller_ccw" value="package://blimp_description/meshes/blimp_propeller/blimp_left_propeller_ccw_v3.dae" />
-  <xacro:property name="mesh_file_bot_propeller_cw" value="package://blimp_description/meshes/blimp_propeller/blimp_bot_propeller_cw_v3.dae" />
-  <xacro:property name="mesh_file_blimp_rud_part1" value="package://blimp_description/meshes/blimp_fin/blimp_top_rud_part1_v3.dae" />
-  <xacro:property name="mesh_file_blimp_rud_part2" value="package://blimp_description/meshes/blimp_fin/blimp_top_rud_part2_v5.dae" />
-  <xacro:property name="mesh_file_blimp_bot_rud_part1" value="package://blimp_description/meshes/blimp_fin/blimp_bot_rud_part1_v3.dae" />
+  <xacro:property name="mesh_file_blimp_body" value="file://$(find blimp_description)/meshes/blimp_body/blimp_body_v4.dae" />
+  <xacro:property name="mesh_file_blimp_support" value="file://$(find blimp_description)/meshes/blimp_support/blimp_support_v5.dae" />
+  <xacro:property name="mesh_file_blimp_gondola" value="file://$(find blimp_description)/meshes/blimp_gondola/blimp_gondola_v4.dae" />
+  <xacro:property name="mesh_file_blimp_wing" value="file://$(find blimp_description)/meshes/blimp_wing/blimp_wing_v2.dae" />
+  <xacro:property name="mesh_file_blimp_stick" value="file://$(find blimp_description)/meshes/blimp_wing/blimp_stick_v2.dae" />
+  <xacro:property name="mesh_file_propeller_cw" value="file://$(find blimp_description)/meshes/blimp_propeller/blimp_right_propeller_cw_v3.dae" />
+  <xacro:property name="mesh_file_propeller_ccw" value="file://$(find blimp_description)/meshes/blimp_propeller/blimp_left_propeller_ccw_v3.dae" />
+  <xacro:property name="mesh_file_bot_propeller_cw" value="file://$(find blimp_description)/meshes/blimp_propeller/blimp_bot_propeller_cw_v3.dae" />
+  <xacro:property name="mesh_file_blimp_rud_part1" value="file://$(find blimp_description)/meshes/blimp_fin/blimp_top_rud_part1_v3.dae" />
+  <xacro:property name="mesh_file_blimp_rud_part2" value="file://$(find blimp_description)/meshes/blimp_fin/blimp_top_rud_part2_v5.dae" />
+  <xacro:property name="mesh_file_blimp_bot_rud_part1" value="file://$(find blimp_description)/meshes/blimp_fin/blimp_bot_rud_part1_v3.dae" />
   <!-- Volume and gas properties -->
   <xacro:property name="volume_total" value="${volume_blimp_body}" />

File: src/blimp_description/urdf/plugin_control.xacro (robot description, xacro)
@@ -11,5 +11,5 @@
       max_rot_velocity motor_number rotor_drag_coefficient
       rolling_moment_coefficient">
-    <!-- Gazebo Harmonic Multicopter Motor Model Plugin - COMPLETELY FIXED -->
+    <!-- Gazebo Harmonic Multicopter Motor Model Plugin - FIXED: Correct filename -->
     <gazebo>
       <plugin filename="gz-sim-multicopter-motor-model-system"
@@ -56,5 +56,5 @@
     </transmission>
   </xacro:macro>
-  <!-- ROS2 Control Hardware Interface -->
+  <!-- ROS2 Control Hardware Interface - FIXED: Correct structure -->
   <xacro:macro name="ros2_control_interface" params="namespace">
     <ros2_control name="${namespace}_control" type="system">
@@ -109,14 +109,4 @@
       </joint>
     </ros2_control>
-    <!-- Gazebo ROS2 Control Plugin - FIXED -->
-    <gazebo>
-      <plugin filename="gz_ros2_control-system"
-              name="gz_ros2_control::GazeboSimROS2ControlPlugin">
-        <parameters>$(find blimp_description)/resource/controller_blimp.yaml</parameters>
-        <ros>
-          <namespace>${namespace}</namespace>
-        </ros>
-      </plugin>
-    </gazebo>
   </xacro:macro>
   <!-- =============================================================== -->
