Commit message: Added PX4 sitl

File: src/blimp_description/urdf/blimp_base.xacro (robot description, xacro)
@@ -33,4 +33,5 @@
   <!--*****************  physics and extra plugins description  *****************-->
   <xacro:include filename="$(find blimp_description)/urdf/description_plugin.xacro"/>
+  <!-- REMOVED: Duplicate Mavlink plugin definition - now handled in description_sensor.xacro -->
   <!-- ROS 2 Control hardware interface (Gazebo Harmonic) -->
   <gazebo>

File: src/blimp_description/urdf/description_plugin.xacro (robot description, xacro)
@@ -4,5 +4,5 @@
   <xacro:if value="$(arg enable_wind)">
     <gazebo>
-      <!-- FIXED: Correct Gazebo Harmonic plugin filename format -->
+      <!-- FIXED: Correct plugin name to match registration -->
       <plugin filename="normwind_plugin" name="normwind_plugin::NormWindPlugin">
         <robotNamespace>${namespace}</robotNamespace>
@@ -23,6 +23,6 @@
     <!-- Main body aerodynamics -->
     <gazebo>
-      <!-- FIXED: Correct Gazebo Harmonic plugin filename format -->
-      <plugin name="blimp_body_finliftdrag" filename="finliftdrag_plugin">
+      <!-- FIXED: Correct plugin name to match registration -->
+      <plugin name="finliftdrag_plugin::FinLiftDragPlugin" filename="finliftdrag_plugin">
         <robotNamespace>${namespace}</robotNamespace>
         <link_name>blimp_body_link</link_name>
@@ -46,6 +46,6 @@
     <!-- Bottom rudder aerodynamics -->
     <gazebo>
-      <!-- FIXED: Correct Gazebo Harmonic plugin filename format -->
-      <plugin name="bot_rud_finliftdrag" filename="finliftdrag_plugin">
+      <!-- FIXED: Correct plugin name to match registration -->
+      <plugin name="finliftdrag_plugin::FinLiftDragPlugin" filename="finliftdrag_plugin">
         <robotNamespace>${namespace}</robotNamespace>
         <link_name>bot_rud_part1_link</link_name>
@@ -71,6 +71,6 @@
     <!-- Top rudder aerodynamics -->
     <gazebo>
-      <!-- FIXED: Correct Gazebo Harmonic plugin filename format -->
-      <plugin name="top_rud_finliftdrag" filename="finliftdrag_plugin">
+      <!-- FIXED: Correct plugin name to match registration -->
+      <plugin name="finliftdrag_plugin::FinLiftDragPlugin" filename="finliftdrag_plugin">
         <robotNamespace>${namespace}</robotNamespace>
         <link_name>top_rud_part1_link</link_name>
@@ -94,12 +94,12 @@
   <xacro:if value="$(arg enable_custom_plugins)">
     <gazebo>
-      <!-- FIXED: Correct Gazebo Harmonic plugin filename format -->
-      <plugin name="dynamicvolume_plugin" filename="dynamicvolume_plugin">
+      <!-- FIXED: Correct plugin name to match registration -->
+      <plugin name="dynamicvolume_plugin::DynamicVolumePlugin" filename="dynamicvolume_plugin">
         <robotNamespace>${namespace}</robotNamespace>
         <linkName>blimp_body_link</linkName>
         <dynamicVolumeTopic>dynamic_volume</dynamicVolumeTopic>
         <heliumMassTopic>helium_mass</heliumMassTopic>
-        <heliumMassKG>1.0</heliumMassKG>
-        <refAlt>0</refAlt>
+        <heliumMassKG>1.723</heliumMassKG>
+        <refAlt>341.0</refAlt>
         <fluidDensity>1.2041</fluidDensity>
         <frameId>world</frameId>
@@ -166,5 +166,5 @@
     <!-- Bottom rudder motor -->
     <gazebo>
-      <!-- FIXED: Correct Gazebo Harmonic built-in plugin filename -->
+      <!-- Correct Gazebo Harmonic built-in plugin filename -->
       <plugin filename="gz-sim-multicopter-motor-model-system"
               name="gz::sim::systems::MulticopterMotorModel">
@@ -190,5 +190,5 @@
     </gazebo>
   </xacro:if>
-  <!-- Ground Truth Odometry - This doesn't reference a specific sensor link -->
+  <!-- Ground Truth Odometry -->
   <xacro:if value="$(arg enable_ground_truth)">
     <gazebo>
@@ -206,3 +206,10 @@
     </gazebo>
   </xacro:if>
+  <!-- PX4 Integration - REMOVED broken plugin, using native GZ bridge instead -->
+  <!-- PX4 automatically connects to sensors when PX4_GZ_MODEL_NAME environment variable is set -->
+  <!-- This eliminates the need for the problematic gz-sim-multicopter-velocity-control-system plugin -->
+  <xacro:if value="$(arg enable_mavlink_interface)">
+    <!-- PX4 native integration enabled via environment variables in launch file -->
+    <!-- No additional plugins needed - PX4 gz_bridge handles sensor integration automatically -->
+  </xacro:if>
 </robot>

File: src/blimp_description/urdf/description_sensor.xacro (robot description, xacro)
@@ -1,32 +1,22 @@
 <?xml version="1.0" ?>
 <robot xmlns:xacro="http://ros.org/wiki/xacro">
-<!--TODO: add compass -->
-<!--TODO: add Gimbal Camera -->
-  <!-- ground truth imu and odo -->
-  <xacro:if value="$(arg enable_ground_truth)">
+  <!-- ✅ SIMPLIFIED: Only essential sensors for PX4 (remove duplicates) -->
+  <!-- ❌ DISABLED: Ground truth sensors (causing PX4 confusion) -->
+  <!-- <xacro:if value="$(arg enable_ground_truth)">
      <xacro:ground_truth_imu_and_odometry namespace="${namespace}" parent_link="base_link" />
+  </xacro:if> -->
+  <xacro:if value="$(arg enable_sensors)">
+    <!-- ✅ ONLY ESSENTIAL PX4 SENSORS (single instance each on base_link) -->
+    <!-- Main IMU for flight control -->
+    <xacro:default_imu namespace="${namespace}" parent_link="base_link" />
+    <!-- Magnetometer for heading estimation -->
+    <xacro:default_magnetometer namespace="${namespace}" parent_link="base_link" />
+    <!-- Barometer for altitude estimation -->
+    <xacro:default_pressure_sensor namespace="${namespace}" parent_link="base_link" />
+    <!-- GPS for navigation -->
+    <xacro:default_gps namespace="${namespace}" parent_link="base_link" />
   </xacro:if>
-  <xacro:if value="$(arg enable_sensors)">
-    <!-- Mount an ADIS16448 IMU. -->
-    <!--<xacro:default_imu namespace="${namespace}" parent_link="top_rud_part1_link" />-->
-    <!-- Mount a GPS. -->
-    <xacro:default_gps namespace="${namespace}" parent_link="top_rud_part1_link" />
-    <!-- more odometry -->
-     <xacro:tail_imu_and_odometry namespace="${namespace}" parent_link="top_rud_part1_link" />
-  </xacro:if>
-  <xacro:if value="$(arg enable_sensors)">
-    <!-- Mount a VI CAMERA. -->
-    <!-- TODO measure weight, xyz of camera -->
-    <xacro:property name="origin_camera">
-      <origin xyz="0.5  0  -0.1" rpy="0  0.7853  0"/>
-    </xacro:property>
-    <!--<xacro:vi_sensor_camera_macro
-      namespace="${namespace}"
-      parent_link="gondola_body_link"
-      mass="0.425"
-      camera_suffix="1"
-      frame_rate="60">
-      <xacro:insert_block name="origin_camera" />
-    </xacro:vi_sensor_camera_macro>-->
+  <!-- ❌ DISABLED: Camera with IMU (causing sensor conflicts) -->
+  <!-- <xacro:if value="$(arg enable_sensors)">
     <xacro:include filename="$(find blimp_description)/urdf/asus_camera.urdf.xacro" />
     <xacro:asus_camera
@@ -36,4 +26,4 @@
         <origin xyz="0.18 0.0 0.07" rpy="0 0.7853 0"/>
     </xacro:asus_camera>
-  </xacro:if>
+  </xacro:if> -->
 </robot>

File: src/blimp_description/urdf/plugin_component_snippets.xacro (robot description, xacro)
@@ -268,107 +268,17 @@
   </xacro:macro>
   <!-- =============================================================== -->
-  <!-- ==================== MAGNETOMETER MACRO ===================== -->
-  <!-- =============================================================== -->
-  <xacro:macro name="magnetometer_plugin_macro"
-    params="namespace magnetometer_suffix parent_link magnetometer_topic
-      mass_magnetometer_sensor ref_mag_north ref_mag_east ref_mag_down
-      noise_normal noise_uniform_initial_bias *inertia *origin">
-    <!-- Magnetometer link -->
-    <link name="magnetometer${magnetometer_suffix}_link">
-      <inertial>
-        <xacro:insert_block name="inertia" />
-        <mass value="${mass_magnetometer_sensor}" />
-        <origin xyz="0 0 0" rpy="0 0 0" />
-      </inertial>
-    </link>
-    <!-- Magnetometer joint -->
-    <joint name="magnetometer${magnetometer_suffix}_joint" type="revolute">
-      <xacro:insert_block name="origin" />
-      <parent link="${parent_link}" />
-      <child link="magnetometer${magnetometer_suffix}_link" />
-      <limit upper="0" lower="0" effort="0" velocity="0" />
-    </joint>
-    <!-- Gazebo Harmonic magnetometer sensor -->
-    <gazebo reference="magnetometer${magnetometer_suffix}_link">
-      <sensor name="magnetometer${magnetometer_suffix}" type="magnetometer">
-        <always_on>true</always_on>
-        <update_rate>100</update_rate>
-        <magnetometer>
-          <x>
-            <noise type="gaussian">
-              <mean>0.0</mean>
-              <stddev>0.000000080</stddev>
-              <bias_mean>0.000000400</bias_mean>
-              <bias_stddev>0.000000400</bias_stddev>
-            </noise>
-          </x>
-          <y>
-            <noise type="gaussian">
-              <mean>0.0</mean>
-              <stddev>0.000000080</stddev>
-              <bias_mean>0.000000400</bias_mean>
-              <bias_stddev>0.000000400</bias_stddev>
-            </noise>
-          </y>
-          <z>
-            <noise type="gaussian">
-              <mean>0.0</mean>
-              <stddev>0.000000080</stddev>
-              <bias_mean>0.000000400</bias_mean>
-              <bias_stddev>0.000000400</bias_stddev>
-            </noise>
-          </z>
-        </magnetometer>
-        <plugin filename="gz-sim-magnetometer-system" name="gz::sim::systems::Magnetometer">
-          <ros>
-            <namespace>${namespace}</namespace>
-            <remapping>~/out:=${magnetometer_topic}</remapping>
-          </ros>
-        </plugin>
-      </sensor>
-    </gazebo>
-  </xacro:macro>
-  <!-- =============================================================== -->
-  <!-- ==================== PRESSURE SENSOR MACRO ================== -->
-  <!-- =============================================================== -->
-  <xacro:macro name="pressure_sensor_plugin_macro"
-    params="namespace pressure_sensor_suffix parent_link pressure_topic
-      mass_pressure_sensor reference_altitude pressure_variance *inertia *origin">
-    <!-- Pressure sensor link -->
-    <link name="pressure_sensor${pressure_sensor_suffix}_link">
-      <inertial>
-        <xacro:insert_block name="inertia" />
-        <mass value="${mass_pressure_sensor}" />
-        <origin xyz="0 0 0" rpy="0 0 0" />
-      </inertial>
-    </link>
-    <!-- Pressure sensor joint -->
-    <joint name="pressure_sensor${pressure_sensor_suffix}_joint" type="revolute">
-      <xacro:insert_block name="origin" />
-      <parent link="${parent_link}" />
-      <child link="pressure_sensor${pressure_sensor_suffix}_link" />
-      <limit upper="0" lower="0" effort="0" velocity="0" />
-    </joint>
-    <!-- Gazebo Harmonic air pressure sensor -->
-    <gazebo reference="pressure_sensor${pressure_sensor_suffix}_link">
-      <sensor name="air_pressure${pressure_sensor_suffix}" type="air_pressure">
-        <always_on>true</always_on>
-        <update_rate>50</update_rate>
-        <air_pressure>
-          <reference_altitude>${reference_altitude}</reference_altitude>
-          <noise type="gaussian">
-            <mean>0.0</mean>
-            <stddev>${pressure_variance}</stddev>
-          </noise>
-        </air_pressure>
-        <plugin filename="gz-sim-air-pressure-system" name="gz::sim::systems::AirPressure">
-          <ros>
-            <namespace>${namespace}</namespace>
-            <remapping>~/out:=${pressure_topic}</remapping>
-          </ros>
-        </plugin>
-      </sensor>
-    </gazebo>
-  </xacro:macro>
+  <!-- ======= REMOVED: Duplicate sensor macros causing conflicts ==== -->
+  <!-- =============================================================== -->
+  <!--
+  ❌ REMOVED to fix sensor duplication:
+  - magnetometer_plugin_macro (now only in plugin_sensors.xacro)
+  - pressure_sensor_plugin_macro (now only in plugin_sensors.xacro)
+  - default_gps (now only in plugin_sensors.xacro)
+  - default_magnetometer (now only in plugin_sensors.xacro)
+  - default_pressure_sensor (now only in plugin_sensors.xacro)
+  These macros were causing duplicate sensor creation which confused PX4's
+  sensor discovery mechanism. Now all sensor macros are centralized in
+  plugin_sensors.xacro to avoid conflicts.
+  -->
   <!-- =============================================================== -->
   <!-- ==================== VI SENSOR MACROS ======================= -->
@@ -568,51 +478,3 @@
     </xacro:imu_plugin_macro>
   </xacro:macro>
-  <!-- =============================================================== -->
-  <!-- ==================== CONVENIENCE MACROS ===================== -->
-  <!-- =============================================================== -->
-  <xacro:macro name="default_gps" params="namespace parent_link">
-    <xacro:gps_plugin_macro
-      namespace="${namespace}"
-      gps_suffix=""
-      parent_link="${parent_link}"
-      gps_topic="gps"
-      ground_speed_topic="ground_speed"
-      mass_gps_sensor="0.015"
-      horizontal_pos_std_dev="3.0"
-      vertical_pos_std_dev="6.0"
-      horizontal_vel_std_dev="0.1"
-      vertical_vel_std_dev="0.1">
-      <inertia ixx="0.00001" ixy="0.0" ixz="0.0" iyy="0.00001" iyz="0.0" izz="0.00001" />
-      <origin xyz="0 0 0" rpy="0 0 0" />
-    </xacro:gps_plugin_macro>
-  </xacro:macro>
-  <xacro:macro name="default_magnetometer" params="namespace parent_link">
-    <xacro:magnetometer_plugin_macro
-      namespace="${namespace}"
-      magnetometer_suffix=""
-      parent_link="${parent_link}"
-      magnetometer_topic="magnetic_field"
-      mass_magnetometer_sensor="0.015"
-      ref_mag_north="0.000021493"
-      ref_mag_east="0.000000815"
-      ref_mag_down="0.000042795"
-      noise_normal="0.000000080 0.000000080 0.000000080"
-      noise_uniform_initial_bias="0.000000400 0.000000400 0.000000400">
-      <inertia ixx="0.00001" ixy="0.0" ixz="0.0" iyy="0.00001" iyz="0.0" izz="0.00001" />
-      <origin xyz="0 0 0" rpy="0 0 0" />
-    </xacro:magnetometer_plugin_macro>
-  </xacro:macro>
-  <xacro:macro name="default_pressure_sensor" params="namespace parent_link">
-    <xacro:pressure_sensor_plugin_macro
-      namespace="${namespace}"
-      pressure_sensor_suffix=""
-      parent_link="${parent_link}"
-      pressure_topic="air_pressure"
-      mass_pressure_sensor="0.015"
-      reference_altitude="500.0"
-      pressure_variance="0.0">
-      <inertia ixx="0.00001" ixy="0.0" ixz="0.0" iyy="0.00001" iyz="0.0" izz="0.00001" />
-      <origin xyz="0 0 0" rpy="0 0 0" />
-    </xacro:pressure_sensor_plugin_macro>
-  </xacro:macro>
 </robot>
