Commit message: Fixed Motor Parameters

File: src/blimp_description/urdf/asus_camera.urdf.xacro (robot description, xacro)
@@ -1,10 +1,32 @@
 <?xml version="1.0"?>
 <robot xmlns:xacro="http://ros.org/wiki/xacro">
-  <!-- Constants -->
-  <xacro:property name="M_PI" value="3.1415926535897931" />
-  <!-- ASUS Xtion camera macro for ROS2/Gazebo Harmonic -->
-  <!-- Preserves all original ROS1 properties while modernizing plugins -->
-  <xacro:macro name="asus_camera" params="name parent namespace *origin">
-    <!-- Main camera joint -->
+  <!-- FIXED: Asus Camera Macro for Gazebo Harmonic -->
+  <xacro:macro name="asus_camera" params="name parent *origin">
+    <!-- Camera Link -->
+    <link name="${name}_link">
+      <inertial>
+        <mass value="0.564"/>
+        <origin xyz="0 0 0" rpy="0 0 0"/>
+        <inertia ixx="0.003881243" ixy="0.0" ixz="0.0"
+                 iyy="0.000498940" iyz="0.0"
+                 izz="0.003879257"/>
+      </inertial>
+      <visual>
+        <origin xyz="0 0 0" rpy="0 0 0"/>
+        <geometry>
+          <box size="0.073 0.276 0.072"/>
+        </geometry>
+        <material name="dark_grey">
+          <color rgba="0.3 0.3 0.3 1.0"/>
+        </material>
+      </visual>
+      <collision>
+        <origin xyz="0 0 0" rpy="0 0 0"/>
+        <geometry>
+          <box size="0.073 0.276 0.072"/>
+        </geometry>
+      </collision>
+    </link>
+    <!-- Camera Joint -->
     <joint name="${name}_joint" type="fixed">
       <xacro:insert_block name="origin"/>
@@ -12,125 +34,84 @@
       <child link="${name}_link"/>
     </joint>
-    <!-- Main camera link - FIXED: Original ROS1 properties -->
-    <link name="${name}_link">
-      <inertial>
-        <!-- FIXED: Original ROS1 mass -->
-        <mass value="0.200" />
-        <origin xyz="0 0 0" rpy="0 0 0" />
-        <!-- FIXED: Original ROS1 inertia values -->
-        <inertia ixx="5.8083e-4" ixy="0" ixz="0" iyy="3.0833e-5" iyz="0" izz="5.9083e-4" />
-      </inertial>
-      <!-- FIXED: Camera is invisible (commented in original ROS1) -->
-      <!--<visual>
-        <origin xyz="0 0 0" rpy="0 0 0" />
-        <geometry>
-          <mesh filename="model://kinect/meshes/kinect.dae"/>
-        </geometry>
-      </visual>-->
-      <collision>
-        <origin xyz="0 0 0" rpy="0 0 0" />
-        <geometry>
-          <!-- FIXED: Original ROS1 collision geometry -->
-          <box size="0.035 0.185 0.025"/>
-        </geometry>
-      </collision>
-    </link>
-    <!-- FIXED: Missing depth frame structure from ROS1 -->
+    <!-- RGB Camera Frame -->
+    <link name="${name}_rgb_frame"/>
+    <joint name="${name}_rgb_joint" type="fixed">
+      <origin xyz="0.0 -0.02 0.0" rpy="0 0 0"/>
+      <parent link="${name}_link"/>
+      <child link="${name}_rgb_frame"/>
+    </joint>
+    <!-- RGB Camera Optical Frame -->
+    <link name="${name}_rgb_optical_frame"/>
+    <joint name="${name}_rgb_optical_joint" type="fixed">
+      <origin xyz="0 0 0" rpy="-1.5708 0 -1.5708"/>
+      <parent link="${name}_rgb_frame"/>
+      <child link="${name}_rgb_optical_frame"/>
+    </joint>
+    <!-- Depth Camera Frame -->
+    <link name="${name}_depth_frame"/>
     <joint name="${name}_depth_joint" type="fixed">
-      <origin xyz="0.0 0.049 0.0" rpy="0 0 0" />
-      <parent link="${name}_link" />
+      <origin xyz="0.0 -0.02 0.0" rpy="0 0 0"/>
+      <parent link="${name}_link"/>
       <child link="${name}_depth_frame"/>
     </joint>
-    <link name="${name}_depth_frame"/>
+    <!-- Depth Camera Optical Frame -->
+    <link name="${name}_depth_optical_frame"/>
     <joint name="${name}_depth_optical_joint" type="fixed">
-      <origin xyz="0 0 0" rpy="${-M_PI/2} 0.0 ${-M_PI/2}" />
-      <parent link="${name}_depth_frame" />
+      <origin xyz="0 0 0" rpy="-1.5708 0 -1.5708"/>
+      <parent link="${name}_depth_frame"/>
       <child link="${name}_depth_optical_frame"/>
     </joint>
-    <link name="${name}_depth_optical_frame"/>
-    <!-- FIXED: Missing RGB frame structure from ROS1 -->
-    <joint name="${name}_rgb_joint" type="fixed">
-      <origin xyz="0.0 0.022 0.0" rpy="0 0 0" />
-      <parent link="${name}_link" />
-      <child link="${name}_rgb_frame"/>
-    </joint>
-    <link name="${name}_rgb_frame"/>
-    <joint name="${name}_rgb_optical_joint" type="fixed">
-      <origin xyz="0 0 0" rpy="${-M_PI/2} 0.0 ${-M_PI/2}" />
-      <parent link="${name}_rgb_frame" />
-      <child link="${name}_rgb_optical_frame"/>
-    </joint>
-    <link name="${name}_rgb_optical_frame"/>
-    <!-- ASUS Xtion PRO camera sensor - FIXED: All original ROS1 properties -->
-    <gazebo reference="${name}_depth_frame">
-      <sensor type="depth" name="${name}">
-        <!-- FIXED: Original ROS1 update rate -->
-        <update_rate>60</update_rate>
+    <!-- Gazebo Harmonic Camera Plugin - CORRECTED -->
+    <gazebo reference="${name}_link">
+      <!-- RGB Camera -->
+      <sensor name="${name}_rgb_camera" type="camera">
         <camera>
-          <!-- FIXED: Original ROS1 FOV (69.5 degrees) -->
-          <horizontal_fov>${69.5 * M_PI/180.0}</horizontal_fov>
+          <horizontal_fov>1.047</horizontal_fov>
           <image>
+            <width>640</width>
+            <height>480</height>
             <format>R8G8B8</format>
-            <!-- FIXED: Original ROS1 high resolution -->
-            <width>2040</width>
-            <height>1086</height>
           </image>
           <clip>
-            <!-- FIXED: Original ROS1 near clip distance -->
-            <near>0.5</near>
+            <near>0.1</near>
             <far>100</far>
           </clip>
         </camera>
-        <!-- Modern ROS2/Gazebo Harmonic plugin replacing libgazebo_ros_openni_kinect.so -->
-        <plugin filename="gz-sim-depth-camera-system" name="gz::sim::systems::DepthCamera">
+        <always_on>1</always_on>
+        <update_rate>30</update_rate>
+        <visualize>true</visualize>
+        <!-- FIXED: Correct plugin filename for Gazebo Harmonic -->
+        <plugin filename="libgz-sim-sensors-system.so" name="gz::sim::systems::Sensors">
           <ros>
-            <remapping>~/image:=${name}/rgb/image_raw</remapping>
-            <remapping>~/depth_image:=${name}/depth/image_raw</remapping>
-            <remapping>~/camera_info:=${name}/rgb/camera_info</remapping>
-            <remapping>~/depth_camera_info:=${name}/depth/camera_info</remapping>
-            <remapping>~/point_cloud:=${name}/depth/points</remapping>
-          </ros>
-          <!-- FIXED: Original ROS1 parameters -->
-          <always_on>true</always_on>
-          <update_rate>60</update_rate>
-          <frame_name>${name}_depth_optical_frame</frame_name>
-          <point_cloud_cutoff>0.6</point_cloud_cutoff>
-          <!-- FIXED: Original ROS1 distortion parameters -->
-          <distortion_k1>0.0</distortion_k1>
-          <distortion_k2>0.0</distortion_k2>
-          <distortion_k3>0.0</distortion_k3>
-          <distortion_t1>0.0</distortion_t1>
-          <distortion_t2>0.0</distortion_t2>
-        </plugin>
-      </sensor>
-    </gazebo>
-    <!-- Additional RGB camera sensor for better ROS2 compatibility -->
-    <gazebo reference="${name}_rgb_frame">
-      <sensor name="${name}_rgb" type="camera">
-        <always_on>true</always_on>
-        <update_rate>60</update_rate>
-        <camera>
-          <horizontal_fov>${69.5 * M_PI/180.0}</horizontal_fov>
-          <image>
-            <width>2040</width>
-            <height>1086</height>
-            <format>R8G8B8</format>
-          </image>
-          <clip>
-            <near>0.5</near>
-            <far>100</far>
-          </clip>
-          <noise>
-            <type>gaussian</type>
-            <mean>0.0</mean>
-            <stddev>0.007</stddev>
-          </noise>
-        </camera>
-        <plugin filename="gz-sim-camera-system" name="gz::sim::systems::Camera">
-          <ros>
+            <namespace></namespace>
             <remapping>~/image:=${name}/rgb/image_raw</remapping>
             <remapping>~/camera_info:=${name}/rgb/camera_info</remapping>
           </ros>
-          <frame_name>${name}_rgb_optical_frame</frame_name>
+        </plugin>
+      </sensor>
+      <!-- Depth Camera -->
+      <sensor name="${name}_depth_camera" type="depth_camera">
+        <camera>
+          <horizontal_fov>1.047</horizontal_fov>
+          <image>
+            <width>640</width>
+            <height>480</height>
+          </image>
+          <clip>
+            <near>0.1</near>
+            <far>100</far>
+          </clip>
+        </camera>
+        <always_on>1</always_on>
+        <update_rate>30</update_rate>
+        <visualize>true</visualize>
+        <!-- FIXED: Correct plugin filename for Gazebo Harmonic -->
+        <plugin filename="libgz-sim-sensors-system.so" name="gz::sim::systems::Sensors">
+          <ros>
+            <namespace></namespace>
+            <remapping>~/image_depth:=${name}/depth/image_raw</remapping>
+            <remapping>~/points:=${name}/depth/points</remapping>
+            <remapping>~/camera_info:=${name}/depth/camera_info</remapping>
+          </ros>
         </plugin>
       </sensor>

File: src/blimp_description/urdf/description_link.xacro (robot description, xacro)
@@ -99,5 +99,7 @@
           <child link="stick_link" />
     <axis xyz="0 0 -1" />
-    <limit effort="${effort_stick}" velocity="${velocity_stick}" lower="${-max_angle_stick}" upper="${max_angle_stick}" />
+    <!-- <limit effort="${effort_stick}" velocity="${velocity_stick}" lower="${-max_angle_stick}" upper="${max_angle_stick}" />  -->
+    <limit lower="0.0" upper="0.0" effort="1000" velocity="0"/>
+    <dynamics damping="5.0"/>
       </joint>
   <!-- Wings -->

File: src/blimp_description/urdf/description_plugin.xacro (robot description, xacro)
@@ -125,10 +125,10 @@
         <actuator_number>0</actuator_number>
         <turningDirection>ccw</turningDirection>
-        REMOVED: <commandSubTopic>command/motor_speed</commandSubTopic>
+        <commandSubTopic>command/motor_speed</commandSubTopic>
         <motorSpeedPubTopic>motor_speed/0</motorSpeedPubTopic>
-        <motorConstant>9.9865e-06</motorConstant>         <!-- Keep original physics -->
+        <motorConstant>${motor_constant}</motorConstant>         <!-- Keep original physics -->
         <momentConstant>0.016</momentConstant>
-        <timeConstantUp>0.0125</timeConstantUp>
-        <timeConstantDown>0.025</timeConstantDown>
+        <timeConstantUp>${time_constant_up}</timeConstantUp>
+        <timeConstantDown>${time_constant_down}</timeConstantDown>
         <maxRotVelocity>838</maxRotVelocity>               <!-- Plugin will scale to this -->
         <motorType>velocity</motorType>
@@ -142,10 +142,10 @@
         <actuator_number>1</actuator_number>
         <turningDirection>cw</turningDirection>
-        REMOVED: <commandSubTopic>command/motor_speed</commandSubTopic>
+        <commandSubTopic>command/motor_speed</commandSubTopic>
         <motorSpeedPubTopic>motor_speed/1</motorSpeedPubTopic>
-        <motorConstant>9.9865e-06</motorConstant>
+        <motorConstant>${motor_constant}</motorConstant>
         <momentConstant>0.016</momentConstant>
-        <timeConstantUp>0.0125</timeConstantUp>
-        <timeConstantDown>0.025</timeConstantDown>
+        <timeConstantUp>${time_constant_up}</timeConstantUp>
+        <timeConstantDown>${time_constant_down}</timeConstantDown>
         <maxRotVelocity>838</maxRotVelocity>
         <motorType>velocity</motorType>
@@ -159,10 +159,10 @@
         <actuator_number>2</actuator_number>
         <turningDirection>cw</turningDirection>
-        REMOVED: <commandSubTopic>command/motor_speed</commandSubTopic>
+        <commandSubTopic>command/motor_speed</commandSubTopic>
         <motorSpeedPubTopic>motor_speed/2</motorSpeedPubTopic>
-        <motorConstant>9.9865e-06</motorConstant>
+        <motorConstant>${motor_constant}</motorConstant>
         <momentConstant>0.016</momentConstant>
-        <timeConstantUp>0.0125</timeConstantUp>
-        <timeConstantDown>0.025</timeConstantDown>
+        <timeConstantUp>${time_constant_up}</timeConstantUp>
+        <timeConstantDown>${time_constant_down}</timeConstantDown>
         <maxRotVelocity>838</maxRotVelocity>
         <motorType>velocity</motorType>

File: src/blimp_description/urdf/description_property.xacro (robot description, xacro)
@@ -83,5 +83,5 @@
   <xacro:property name="rotor_velocity_slowdown_sim" value="1" />
   <xacro:property name="rotor_offset_top" value="0.05" /> <!-- [m] -->
-  <xacro:property name="motor_constant" value="9.9865e-06" /> <!-- [kg m/s^2] -->
+  <xacro:property name="motor_constant" value="3.71178707e-03" /> <!-- [kg m/s^2] -->
   <xacro:property name="moment_constant" value="0.016" /> <!-- [m] -->
   <!-- FIXED: Original ROS1 motor time constants for realistic motor dynamics -->
@@ -212,5 +212,6 @@
   </xacro:property>
   <xacro:property name="origin_stick_right_blade_joint">
-    <origin xyz="0.0 0.025 0.375" rpy="${-pi/2} 0.0 ${pi}"/>
+    <!-- <origin xyz="0.0 0.025 0.375" rpy="${-pi/2} 0.0 ${pi}"/> -->
+     <origin xyz="0.0 0.025 0.375" rpy="${-pi/2} 0.0 0.0"/>
   </xacro:property>
   <!-- FIXED: Original ROS1 rudder and elevator positioning -->

File: src/blimp_description/urdf/description_sensor.xacro (robot description, xacro)
@@ -9,4 +9,12 @@
       <xacro:default_magnetometer namespace="${namespace}" parent_link="base_link" />    <!-- Creates mag_sensor -->
   </xacro:if>
+  <xacro:if value="$(arg enable_sensors)">
+		<!-- <xacro:include filename="$(find blimp_description)/urdf/asus_camera.urdf.xacro" />
+		<xacro:asus_camera
+		    name="xtion"
+		    parent="gondola_body_link">
+		    <origin xyz="0.18 0.0 0.07" rpy="0 0.7853 0"/>
+		</xacro:asus_camera> -->
+	</xacro:if>
     <!-- SEPARATE BLOCK: Ground truth only if needed for debugging -->
   <!-- <xacro:if value="$(arg enable_ground_truth)">
