Commit message: Fixing controller/motor plugin

File: src/blimp_description/urdf/description_plugin.xacro (robot description, xacro)
@@ -114,77 +114,57 @@
   <!-- MOTOR PLUGINS - FIXED: Conditional inclusion -->
   <xacro:if value="$(arg enable_physics)">
-    <!-- Left blade motor -->
+    <!-- Right blade motor -->
     <gazebo>
-      <!-- FIXED: Correct Gazebo Harmonic built-in plugin filename -->
+      <!-- CORRECTED: Motor plugins using native Actuators interface -->
+      <!-- Motor 0: Left Blade -->
       <plugin filename="gz-sim-multicopter-motor-model-system"
               name="gz::sim::systems::MulticopterMotorModel">
         <robotNamespace>${namespace}</robotNamespace>
+        <jointName>stick_left_blade_joint</jointName>
         <linkName>left_blade_link</linkName>
-        <jointName>stick_left_blade_joint</jointName>
+        <actuator_number>0</actuator_number>
         <turningDirection>ccw</turningDirection>
+        REMOVED: <commandSubTopic>command/motor_speed</commandSubTopic>
+        <motorSpeedPubTopic>motor_speed/0</motorSpeedPubTopic>
+        <motorConstant>9.9865e-06</motorConstant>         <!-- Keep original physics -->
+        <momentConstant>0.016</momentConstant>
+        <timeConstantUp>0.0125</timeConstantUp>
+        <timeConstantDown>0.025</timeConstantDown>
+        <maxRotVelocity>838</maxRotVelocity>               <!-- Plugin will scale to this -->
+        <motorType>velocity</motorType>
+      </plugin>
+      <!-- Motor 1: Right Blade -->
+      <plugin filename="gz-sim-multicopter-motor-model-system"
+              name="gz::sim::systems::MulticopterMotorModel">
+        <robotNamespace>${namespace}</robotNamespace>
+        <jointName>stick_right_blade_joint</jointName>
+        <linkName>right_blade_link</linkName>
+        <actuator_number>1</actuator_number>
+        <turningDirection>cw</turningDirection>
+        REMOVED: <commandSubTopic>command/motor_speed</commandSubTopic>
+        <motorSpeedPubTopic>motor_speed/1</motorSpeedPubTopic>
+        <motorConstant>9.9865e-06</motorConstant>
+        <momentConstant>0.016</momentConstant>
         <timeConstantUp>0.0125</timeConstantUp>
         <timeConstantDown>0.025</timeConstantDown>
         <maxRotVelocity>838</maxRotVelocity>
-        <motorConstant>8.54858e-06</motorConstant>
-        <momentConstant>0.016</momentConstant>
-        <commandSubTopic>command/motor_speed</commandSubTopic>
-        <actuator_number>0</actuator_number>
-        <rotorDragCoefficient>8.06428e-05</rotorDragCoefficient>
-        <rollingMomentCoefficient>1e-06</rollingMomentCoefficient>
-        <motorSpeedPubTopic>motor_speed/0</motorSpeedPubTopic>
         <motorType>velocity</motorType>
-        <ros>
-          <namespace>${namespace}</namespace>
-        </ros>
       </plugin>
-    </gazebo>
-    <!-- Right blade motor -->
-    <gazebo>
-      <!-- FIXED: Correct Gazebo Harmonic built-in plugin filename -->
+      <!-- Motor 2: Bottom Rudder -->
       <plugin filename="gz-sim-multicopter-motor-model-system"
               name="gz::sim::systems::MulticopterMotorModel">
         <robotNamespace>${namespace}</robotNamespace>
-        <linkName>right_blade_link</linkName>
-        <jointName>stick_right_blade_joint</jointName>
+        <jointName>bot_rud_part1_bot_rud_motor_joint</jointName>
+        <linkName>bot_rud_motor_link</linkName>
+        <actuator_number>2</actuator_number>
         <turningDirection>cw</turningDirection>
+        REMOVED: <commandSubTopic>command/motor_speed</commandSubTopic>
+        <motorSpeedPubTopic>motor_speed/2</motorSpeedPubTopic>
+        <motorConstant>9.9865e-06</motorConstant>
+        <momentConstant>0.016</momentConstant>
         <timeConstantUp>0.0125</timeConstantUp>
         <timeConstantDown>0.025</timeConstantDown>
         <maxRotVelocity>838</maxRotVelocity>
-        <motorConstant>8.54858e-06</motorConstant>
-        <momentConstant>0.016</momentConstant>
-        <commandSubTopic>command/motor_speed</commandSubTopic>
-        <actuator_number>1</actuator_number>
-        <rotorDragCoefficient>8.06428e-05</rotorDragCoefficient>
-        <rollingMomentCoefficient>1e-06</rollingMomentCoefficient>
-        <motorSpeedPubTopic>motor_speed/1</motorSpeedPubTopic>
         <motorType>velocity</motorType>
-        <ros>
-          <namespace>${namespace}</namespace>
-        </ros>
-      </plugin>
-    </gazebo>
-    <!-- Bottom rudder motor -->
-    <gazebo>
-      <!-- Correct Gazebo Harmonic built-in plugin filename -->
-      <plugin filename="gz-sim-multicopter-motor-model-system"
-              name="gz::sim::systems::MulticopterMotorModel">
-        <robotNamespace>${namespace}</robotNamespace>
-        <linkName>bot_rud_motor_link</linkName>
-        <jointName>bot_rud_part1_bot_rud_motor_joint</jointName>
-        <turningDirection>cw</turningDirection>
-        <timeConstantUp>0.0125</timeConstantUp>
-        <timeConstantDown>0.025</timeConstantDown>
-        <maxRotVelocity>838</maxRotVelocity>
-        <motorConstant>8.54858e-06</motorConstant>
-        <momentConstant>0.016</momentConstant>
-        <commandSubTopic>command/motor_speed</commandSubTopic>
-        <actuator_number>2</actuator_number>
-        <rotorDragCoefficient>8.06428e-05</rotorDragCoefficient>
-        <rollingMomentCoefficient>1e-06</rollingMomentCoefficient>
-        <motorSpeedPubTopic>motor_speed/2</motorSpeedPubTopic>
-        <motorType>velocity</motorType>
-        <ros>
-          <namespace>${namespace}</namespace>
-        </ros>
       </plugin>
     </gazebo>

File: src/blimp_description/urdf/description_property.xacro (robot description, xacro)
@@ -83,5 +83,5 @@
   <xacro:property name="rotor_velocity_slowdown_sim" value="1" />
   <xacro:property name="rotor_offset_top" value="0.05" /> <!-- [m] -->
-  <xacro:property name="motor_constant" value="3.71178707e-03" /> <!-- [kg m/s^2] -->
+  <xacro:property name="motor_constant" value="9.9865e-06" /> <!-- [kg m/s^2] -->
   <xacro:property name="moment_constant" value="0.016" /> <!-- [m] -->
   <!-- FIXED: Original ROS1 motor time constants for realistic motor dynamics -->

Commit message: Minor tweaks for simplicity

File: src/blimp_description/urdf/description_plugin.xacro (robot description, xacro)
@@ -178,9 +178,10 @@
         <motorSpeedPubTopic>motor_speed/0</motorSpeedPubTopic>
         <motorConstant>${motor_constant}</motorConstant>         <!-- Keep original physics -->
-        <momentConstant>0.016</momentConstant>
+        <momentConstant>0.</momentConstant>
         <timeConstantUp>${time_constant_up}</timeConstantUp>
         <timeConstantDown>${time_constant_down}</timeConstantDown>
         <maxRotVelocity>838</maxRotVelocity>               <!-- Plugin will scale to this -->
         <motorType>velocity</motorType>
+        <rotorVelocitySlowdownSim>1</rotorVelocitySlowdownSim>
       </plugin>
       <!-- Motor 1: Right Blade -->
@@ -195,9 +196,10 @@
         <motorSpeedPubTopic>motor_speed/1</motorSpeedPubTopic>
         <motorConstant>${motor_constant}</motorConstant>
-        <momentConstant>0.016</momentConstant>
+        <momentConstant>0</momentConstant>
         <timeConstantUp>${time_constant_up}</timeConstantUp>
         <timeConstantDown>${time_constant_down}</timeConstantDown>
         <maxRotVelocity>838</maxRotVelocity>
         <motorType>velocity</motorType>
+        <rotorVelocitySlowdownSim>1</rotorVelocitySlowdownSim>
       </plugin>
       <!-- Motor 2: Bottom Rudder -->
@@ -212,9 +214,10 @@
         <motorSpeedPubTopic>motor_speed/2</motorSpeedPubTopic>
         <motorConstant>${motor_constant}</motorConstant>
-        <momentConstant>0.016</momentConstant>
+        <momentConstant>0</momentConstant>
         <timeConstantUp>${time_constant_up}</timeConstantUp>
         <timeConstantDown>${time_constant_down}</timeConstantDown>
         <maxRotVelocity>838</maxRotVelocity>
         <motorType>velocity</motorType>
+        <rotorVelocitySlowdownSim>1</rotorVelocitySlowdownSim>
       </plugin>
     </gazebo>

File: src/blimp_description/urdf/description_property.xacro (robot description, xacro)
@@ -86,6 +86,6 @@
   <xacro:property name="moment_constant" value="0.016" /> <!-- [m] -->
   <!-- FIXED: Original ROS1 motor time constants for realistic motor dynamics -->
-  <xacro:property name="time_constant_up" value="0.0125" /> <!-- [s] -->
-  <xacro:property name="time_constant_down" value="0.025" /> <!-- [s] -->
+  <xacro:property name="time_constant_up" value="0.05" /> <!-- [s] -->
+  <xacro:property name="time_constant_down" value="0.08" /> <!-- [s] -->
   <xacro:property name="max_rot_velocity" value="879.23" /> <!-- [rad/s] -->
   <xacro:property name="rotor_drag_coefficient" value="8.06428e-05" />
