Commit message: Blimp model fixed

File: src/blimp_description/urdf/description_link.xacro (robot description, xacro)
@@ -228,5 +228,6 @@
     robot_namespace="${namespace}"
                 link_name="top_rud_base_joint"
-                parent="blimp_body_link">
+                parent="blimp_body_link"
+                strength_factor="2">
     <xacro:insert_block name="origin_top_rud_base_link_joint" />
   </xacro:spring>
@@ -250,5 +251,5 @@
       </joint>
   <link name="top_rud_joint_link">
-    <!-- ADDED: Minimal inertial properties required by Gazebo Harmonic (ROS1 had none) -->
+    <!-- FIXED: Proper inertial properties required by Gazebo Harmonic -->
     <inertial>
       <mass value="1e-6"/>
@@ -290,5 +291,6 @@
     robot_namespace="${namespace}"
                 link_name="bot_rud_base_joint"
-                parent="blimp_body_link">
+                parent="blimp_body_link"
+                strength_factor="2">
     <xacro:insert_block name="origin_bot_rud_base_link_joint" />
   </xacro:spring>
@@ -303,5 +305,6 @@
         mesh_file="${mesh_file_blimp_bot_rud_part1}">
     <xacro:insert_block name="origin_rud_part1" />
-    <xacro:insert_block name="inertia_rud_part1" />
+    <!-- FIXED: Use correct separate bot rudder inertia from original ROS1 -->
+    <xacro:insert_block name="inertia_bot_rud_part1" />
   </xacro:box_model>
   <joint name="blimp_body_bot_rud_part1_joint" type="revolute">
@@ -312,5 +315,5 @@
       </joint>
   <link name="bot_rud_joint_link">
-    <!-- ADDED: Minimal inertial properties required by Gazebo Harmonic (ROS1 had none) -->
+    <!-- FIXED: Proper inertial properties required by Gazebo Harmonic -->
     <inertial>
       <mass value="1e-6"/>
@@ -364,5 +367,6 @@
           <parent link="bot_rud_part1_link" />
           <child link="bot_rud_motor_link" />
-    <axis xyz="0 0 1" />
+    <!-- FIXED: Correct axis from original ROS1 implementation -->
+    <axis xyz="0 0 -1" />
       </joint>
   <!-- Left elevator assembly -->
@@ -370,5 +374,6 @@
     robot_namespace="${namespace}"
                 link_name="left_elv_base_joint"
-                parent="blimp_body_link">
+                parent="blimp_body_link"
+                strength_factor="2">
     <xacro:insert_block name="origin_left_elv_base_link_joint" />
   </xacro:spring>
@@ -392,5 +397,5 @@
       </joint>
   <link name="left_elv_joint_link">
-    <!-- ADDED: Minimal inertial properties required by Gazebo Harmonic (ROS1 had none) -->
+    <!-- FIXED: Proper inertial properties required by Gazebo Harmonic -->
     <inertial>
       <mass value="1e-6"/>
@@ -408,5 +413,6 @@
           <parent link="left_elv_part1_link" />
           <child link="left_elv_joint_link" />
-    <axis xyz="0 0 -1" />
+    <!-- FIXED: Correct axis from original ROS1 (was 0 0 -1) -->
+    <axis xyz="0 0 1" />
     <limit effort="${effort_fin}" velocity="${velocity_fin}" lower="${-max_angle_fin}" upper="${max_angle_fin}" />
       </joint>
@@ -432,5 +438,6 @@
     robot_namespace="${namespace}"
                 link_name="right_elv_base_joint"
-                parent="blimp_body_link">
+                parent="blimp_body_link"
+                strength_factor="2">
     <xacro:insert_block name="origin_right_elv_base_link_joint" />
   </xacro:spring>
@@ -454,5 +461,5 @@
       </joint>
   <link name="right_elv_joint_link">
-    <!-- ADDED: Minimal inertial properties required by Gazebo Harmonic (ROS1 had none) -->
+    <!-- FIXED: Proper inertial properties required by Gazebo Harmonic -->
     <inertial>
       <mass value="1e-6"/>

File: src/blimp_description/urdf/description_property.xacro (robot description, xacro)
@@ -85,6 +85,7 @@
   <xacro:property name="motor_constant" value="3.71178707e-03" /> <!-- [kg m/s^2] -->
   <xacro:property name="moment_constant" value="0.016" /> <!-- [m] -->
-  <xacro:property name="time_constant_up" value="1" /> <!-- [s] -->
-  <xacro:property name="time_constant_down" value="1" /> <!-- [s] -->
+  <!-- FIXED: Original ROS1 motor time constants for realistic motor dynamics -->
+  <xacro:property name="time_constant_up" value="0.0125" /> <!-- [s] -->
+  <xacro:property name="time_constant_down" value="0.025" /> <!-- [s] -->
   <xacro:property name="max_rot_velocity" value="879.23" /> <!-- [rad/s] -->
   <xacro:property name="rotor_drag_coefficient" value="8.06428e-05" />
@@ -117,8 +118,8 @@
   </xacro:property>
   <xacro:property name="inertia_wing">
-        <xacro:cylinder_inertia r="${radius_wing}" h="${length_wing}" mass="${mass_wing}"/>
+        <xacro:hollow_cylinder_inertia r1="${radius_wing - length_wing_skin}" r2="${radius_wing}" h="${length_wing}" mass="${mass_wing}"/>
   </xacro:property>
   <xacro:property name="inertia_blade">
-        <xacro:cylinder_inertia r="${radius_blade}" h="${length_blade}" mass="${mass_blade}"/>
+        <xacro:cylinder_inertia r="${radius_blade}" h="${length_blade}" mass="${mass_blade*rotor_velocity_slowdown_sim}"/>
   </xacro:property>
   <xacro:property name="inertia_rud_part1">
@@ -128,6 +129,10 @@
         <xacro:cuboid_inertia x="${length_rud_part2}" y="${width_rud_part2}" z="${height_rud_part2}" mass="${mass_rud_part2}"/>
   </xacro:property>
+  <!-- FIXED: Added missing separate bot rudder part1 inertia from original ROS1 -->
+  <xacro:property name="inertia_bot_rud_part1">
+        <xacro:cuboid_inertia x="${length_rud_part1}" y="${width_rud_part1}" z="${height_rud_part1}" mass="${mass_bot_rud_part1}"/>
+  </xacro:property>
   <xacro:property name="inertia_bot_rud_motor">
-        <xacro:cylinder_inertia r="${radius_bot_rud_motor}" h="${length_bot_rud_motor}" mass="${mass_bot_rud_motor}"/>
+        <xacro:cylinder_inertia r="${radius_bot_rud_motor}" h="${length_bot_rud_motor}" mass="${mass_bot_rud_motor*rotor_velocity_slowdown_sim}"/>
   </xacro:property>
   <xacro:property name="inertia_ballast">
@@ -168,4 +173,5 @@
     <origin xyz="0  0  0" rpy="0  0  0"/>
   </xacro:property>
+  <!-- FIXED: Correct joint origins from original ROS1 implementation -->
   <!-- joint origins [m] [m] [m] [rad] [rad] [rad] -->
   <xacro:property name="origin_blimp_body_forward_lift_joint">
@@ -208,54 +214,55 @@
     <origin xyz="0.0 0.025 0.375" rpy="${-pi/2} 0.0 ${pi}"/>
   </xacro:property>
+  <!-- FIXED: Original ROS1 rudder and elevator positioning -->
   <xacro:property name="origin_top_rud_base_link_joint">
-    <origin xyz="0 0 -2.25" rpy="0.0 0.0 0.0"/>
+    <origin xyz="-0.59 0.0 -1.5" rpy="${pi} ${-pi/2} 0.0"/>
   </xacro:property>
   <xacro:property name="origin_blimp_body_top_rud_part1_joint">
-    <origin xyz="0.0 0.0 0.0" rpy="0.0 0.0 0.0"/>
+    <origin xyz="0.0 0.0 -0.24" rpy="0.0 0.0 0.0"/>
   </xacro:property>
   <xacro:property name="origin_top_rud_part1_top_rud_joint_link_joint">
-    <origin xyz="0.0 0.0 0.0" rpy="0.0 0.0 0.0"/>
+    <origin xyz="-0.28 0.0 0.0" rpy="0.0 0.0 0.0"/>
   </xacro:property>
   <xacro:property name="origin_top_rud_joint_link_top_rud_part2_joint">
-    <origin xyz="0.0 0.0 0.0" rpy="0.0 0.0 0.0"/>
+    <origin xyz="-0.125 0.0 0.0" rpy="0.0 0.0 0.0"/>
   </xacro:property>
   <xacro:property name="origin_bot_rud_base_link_joint">
-    <origin xyz="0 0 2.25" rpy="0.0 0.0 0.0"/>
+    <origin xyz="0.59 0.0 -1.5" rpy="0.0 ${-pi/2} 0.0"/>
   </xacro:property>
   <xacro:property name="origin_blimp_body_bot_rud_part1_joint">
-    <origin xyz="0.0 0.0 0.0" rpy="0.0 0.0 0.0"/>
+    <origin xyz="0.0 0.0 -0.24" rpy="0.0 0.0 0.0"/>
   </xacro:property>
   <xacro:property name="origin_bot_rud_part1_bot_rud_joint_link_joint">
-    <origin xyz="0.0 0.0 0.0" rpy="0.0 0.0 0.0"/>
+    <origin xyz="-0.28 0.0 0.0" rpy="0.0 0.0 0.0"/>
   </xacro:property>
   <xacro:property name="origin_bot_rud_joint_link_bot_rud_part2_joint">
-    <origin xyz="0.0 0.0 0.0" rpy="0.0 0.0 0.0"/>
+    <origin xyz="-0.125 0.0 0.0" rpy="0.0 0.0 0.0"/>
   </xacro:property>
   <xacro:property name="origin_bot_rud_part1_bot_rud_motor_joint">
-    <origin xyz="0.0 0.0 0.3" rpy="0.0 0.0 0.0"/>
+    <origin xyz="-0.065 0.01 -0.025" rpy="${-pi/2} 0.0 0.0"/>
   </xacro:property>
   <xacro:property name="origin_left_elv_base_link_joint">
-    <origin xyz="-0.6 0.8 0.0" rpy="0.0 0.0 ${pi/2}"/>
+    <origin xyz="0.0 0.59 -1.5" rpy="0.0 ${-pi/2} ${pi/2}"/>
   </xacro:property>
   <xacro:property name="origin_blimp_body_left_elv_part1_joint">
-    <origin xyz="0.0 0.0 0.0" rpy="0.0 0.0 0.0"/>
+    <origin xyz="0.0 0.0 -0.24" rpy="0.0 0.0 0.0"/>
   </xacro:property>
   <xacro:property name="origin_left_elv_part1_left_elv_joint_link_joint">
-    <origin xyz="0.0 0.0 0.0" rpy="0.0 0.0 0.0"/>
+    <origin xyz="-0.28 0.0 0.0" rpy="0.0 0.0 0.0"/>
   </xacro:property>
   <xacro:property name="origin_left_elv_joint_link_left_elv_part2_joint">
-    <origin xyz="0.0 0.0 0.0" rpy="0.0 0.0 0.0"/>
+    <origin xyz="-0.125 0.0 0.0" rpy="0.0 0.0 0.0"/>
   </xacro:property>
   <xacro:property name="origin_right_elv_base_link_joint">
-    <origin xyz="-0.6 -0.8 0.0" rpy="0.0 0.0 ${-pi/2}"/>
+    <origin xyz="0.0 -0.59 -1.5" rpy="0.0 ${-pi/2} ${-pi/2}"/>
   </xacro:property>
   <xacro:property name="origin_blimp_body_right_elv_part1_joint">
-    <origin xyz="0.0 0.0 0.0" rpy="0.0 0.0 0.0"/>
+    <origin xyz="0.0 0.0 -0.24" rpy="0.0 0.0 0.0"/>
   </xacro:property>
   <xacro:property name="origin_right_elv_part1_right_elv_joint_link_joint">
-    <origin xyz="0.0 0.0 0.0" rpy="0.0 0.0 0.0"/>
+    <origin xyz="-0.28 0.0 0.0" rpy="0.0 0.0 0.0"/>
   </xacro:property>
   <xacro:property name="origin_right_elv_joint_link_right_elv_part2_joint">
-    <origin xyz="0.0 0.0 0.0" rpy="0.0 0.0 0.0"/>
+    <origin xyz="-0.125 0.0 0.0" rpy="0.0 0.0 0.0"/>
   </xacro:property>
 </robot>

Commit message: Worked on Joint

File: src/blimp_description/urdf/description_link.xacro (robot description, xacro)
@@ -98,9 +98,8 @@
           <parent link="base_link" />
           <child link="stick_link" />
-    <axis xyz="0 0 -1" />
-    <!-- <limit effort="${effort_stick}" velocity="${velocity_stick}" lower="${-max_angle_stick}" upper="${max_angle_stick}" />  -->
-    <limit lower="0.0" upper="0.0" effort="1000" velocity="0"/>
+    <axis xyz="0 0 1" />
+    <limit effort="${effort_stick}" velocity="${velocity_stick}" lower="${-max_angle_stick}" upper="${max_angle_stick}" />
     <dynamics damping="5.0"/>
-      </joint>
+  </joint>
   <!-- Wings -->
   <xacro:cylinder_model
@@ -119,5 +118,5 @@
           <parent link="stick_link" />
           <child link="left_wing_link" />
-      </joint>
+  </joint>
   <xacro:cylinder_model
     robot_namespace="${namespace}"
@@ -135,5 +134,5 @@
           <parent link="stick_link" />
           <child link="right_wing_link" />
-      </joint>
+  </joint>
   <!-- Propeller blades -->
   <xacro:cylinder_model
@@ -153,5 +152,5 @@
           <child link="left_blade_link" />
     <axis xyz="0 0 1" />
-      </joint>
+  </joint>
   <xacro:cylinder_model
     robot_namespace="${namespace}"
@@ -170,5 +169,5 @@
           <child link="right_blade_link" />
     <axis xyz="0 0 1" />
-      </joint>
+  </joint>
   <!-- Ballast weight -->
   <xacro:cylinder_model
@@ -225,5 +224,5 @@
           <child link="aft_lift_joint_link" />
     <limit effort="1000" velocity="1000" lower="0" upper="0" />
-      </joint>
+  </joint>
   <!-- Top rudder assembly -->
   <xacro:spring
@@ -251,5 +250,5 @@
           <child link="top_rud_part1_link" />
     <limit effort="1000" velocity="1000" lower="0" upper="0" />
-      </joint>
+  </joint>
   <link name="top_rud_joint_link">
     <!-- FIXED: Proper inertial properties required by Gazebo Harmonic -->
@@ -271,5 +270,5 @@
     <axis xyz="0 0 -1" />
     <limit effort="${effort_fin}" velocity="${velocity_fin}" lower="${-max_angle_fin}" upper="${max_angle_fin}" />
-      </joint>
+  </joint>
   <xacro:box_model
     robot_namespace="${namespace}"
@@ -288,5 +287,5 @@
           <parent link="top_rud_joint_link" />
           <child link="top_rud_part2_link" />
-      </joint>
+  </joint>
   <!-- Bottom rudder assembly -->
   <xacro:spring
@@ -335,5 +334,5 @@
     <axis xyz="0 0 1" />
     <limit effort="${effort_fin}" velocity="${velocity_fin}" lower="${-max_angle_fin}" upper="${max_angle_fin}" />
-      </joint>
+  </joint>
   <xacro:box_model
     robot_namespace="${namespace}"
@@ -352,5 +351,5 @@
           <parent link="bot_rud_joint_link" />
           <child link="bot_rud_part2_link" />
-      </joint>
+  </joint>
   <!-- Bottom rudder motor -->
   <xacro:cylinder_model
@@ -371,5 +370,5 @@
     <!-- FIXED: Correct axis from original ROS1 implementation -->
     <axis xyz="0 0 -1" />
-      </joint>
+  </joint>
   <!-- Left elevator assembly -->
   <xacro:spring
@@ -397,5 +396,5 @@
           <child link="left_elv_part1_link" />
     <limit effort="1000" velocity="1000" lower="0" upper="0" />
-      </joint>
+  </joint>
   <link name="left_elv_joint_link">
     <!-- FIXED: Proper inertial properties required by Gazebo Harmonic -->
@@ -418,5 +417,5 @@
     <axis xyz="0 0 1" />
     <limit effort="${effort_fin}" velocity="${velocity_fin}" lower="${-max_angle_fin}" upper="${max_angle_fin}" />
-      </joint>
+  </joint>
   <xacro:box_model
     robot_namespace="${namespace}"
@@ -435,5 +434,5 @@
           <parent link="left_elv_joint_link" />
           <child link="left_elv_part2_link" />
-      </joint>
+ </joint>
   <!-- Right elevator assembly -->
   <xacro:spring
@@ -461,5 +460,5 @@
           <child link="right_elv_part1_link" />
     <limit effort="1000" velocity="1000" lower="0" upper="0" />
-      </joint>
+  </joint>
   <link name="right_elv_joint_link">
     <!-- FIXED: Proper inertial properties required by Gazebo Harmonic -->
@@ -481,5 +480,5 @@
     <axis xyz="0 0 1" />
     <limit effort="${effort_fin}" velocity="${velocity_fin}" lower="${-max_angle_fin}" upper="${max_angle_fin}" />
-      </joint>
+  </joint>
   <xacro:box_model
     robot_namespace="${namespace}"
@@ -498,5 +497,5 @@
           <parent link="right_elv_joint_link" />
           <child link="right_elv_part2_link" />
-      </joint>
+  </joint>
 <!-- REMOVED: Hardcoded sensor links - these are now handled by sensor plugin macros -->
 <!-- The following hardcoded sensor links were causing duplicates:

File: src/blimp_description/urdf/description_plugin.xacro (robot description, xacro)
@@ -186,4 +186,15 @@
     </gazebo>
   </xacro:if>
+  <!-- Tilt Joint Controller -->
+  <xacro:if value="$(arg enable_physics)">
+    <gazebo>
+      <plugin filename="gz-sim-joint-position-controller-system"
+              name="gz::sim::systems::JointPositionController">
+        <joint_name>base_stick_joint</joint_name>
+        <sub_topic>servo_0</sub_topic>
+        <p_gain>100</p_gain>
+      </plugin>
+    </gazebo>
+  </xacro:if>
   <!-- PX4 Integration - REMOVED broken plugin, using native GZ bridge instead -->
   <!-- PX4 automatically connects to sensors when PX4_GZ_MODEL_NAME environment variable is set -->

Commit message: Added Servo Scaling

File: src/blimp_description/urdf/description_link.xacro (robot description, xacro)
@@ -98,5 +98,5 @@
           <parent link="base_link" />
           <child link="stick_link" />
-    <axis xyz="0 0 1" />
+    <axis xyz="0 0 -1" />
     <limit effort="${effort_stick}" velocity="${velocity_stick}" lower="${-max_angle_stick}" upper="${max_angle_stick}" />
     <dynamics damping="5.0"/>

File: src/blimp_description/urdf/description_plugin.xacro (robot description, xacro)
@@ -192,5 +192,5 @@
               name="gz::sim::systems::JointPositionController">
         <joint_name>base_stick_joint</joint_name>
-        <sub_topic>servo_0</sub_topic>
+        <sub_topic>servo_0_scaled</sub_topic>  <!-- Scaling by 2 times as PX4 is giving half the angle -->
         <p_gain>100</p_gain>
       </plugin>

Commit message: Thruster tweak

File: src/blimp_description/urdf/description_link.xacro (robot description, xacro)
@@ -414,6 +414,5 @@
           <parent link="left_elv_part1_link" />
           <child link="left_elv_joint_link" />
-    <!-- FIXED: Correct axis from original ROS1 (was 0 0 -1) -->
-    <axis xyz="0 0 1" />
+    <axis xyz="0 0 -1" />
     <limit effort="${effort_fin}" velocity="${velocity_fin}" lower="${-max_angle_fin}" upper="${max_angle_fin}" />
   </joint>

File: src/blimp_description/urdf/description_plugin.xacro (robot description, xacro)
@@ -178,10 +178,10 @@
         <motorSpeedPubTopic>motor_speed/0</motorSpeedPubTopic>
         <motorConstant>${motor_constant}</motorConstant>         <!-- Keep original physics -->
-        <momentConstant>0.</momentConstant>
+        <momentConstant>${moment_constant}</momentConstant>
         <timeConstantUp>${time_constant_up}</timeConstantUp>
         <timeConstantDown>${time_constant_down}</timeConstantDown>
         <maxRotVelocity>838</maxRotVelocity>               <!-- Plugin will scale to this -->
         <motorType>velocity</motorType>
-        <rotorVelocitySlowdownSim>1</rotorVelocitySlowdownSim>
+        <!-- <rotorVelocitySlowdownSim>100</rotorVelocitySlowdownSim> -->
       </plugin>
       <!-- Motor 1: Right Blade -->
@@ -196,28 +196,24 @@
         <motorSpeedPubTopic>motor_speed/1</motorSpeedPubTopic>
         <motorConstant>${motor_constant}</motorConstant>
-        <momentConstant>0</momentConstant>
+        <momentConstant>${moment_constant}</momentConstant>
         <timeConstantUp>${time_constant_up}</timeConstantUp>
         <timeConstantDown>${time_constant_down}</timeConstantDown>
         <maxRotVelocity>838</maxRotVelocity>
         <motorType>velocity</motorType>
-        <rotorVelocitySlowdownSim>1</rotorVelocitySlowdownSim>
-      </plugin>
-      <!-- Motor 2: Bottom Rudder -->
-      <plugin filename="gz-sim-multicopter-motor-model-system"
-              name="gz::sim::systems::MulticopterMotorModel">
-        <robotNamespace>${namespace}</robotNamespace>
-        <jointName>bot_rud_part1_bot_rud_motor_joint</jointName>
-        <linkName>bot_rud_motor_link</linkName>
-        <actuator_number>2</actuator_number>
-        <turningDirection>cw</turningDirection>
-        <commandSubTopic>command/motor_speed</commandSubTopic>
-        <motorSpeedPubTopic>motor_speed/2</motorSpeedPubTopic>
-        <motorConstant>${motor_constant}</motorConstant>
-        <momentConstant>0</momentConstant>
-        <timeConstantUp>${time_constant_up}</timeConstantUp>
-        <timeConstantDown>${time_constant_down}</timeConstantDown>
-        <maxRotVelocity>838</maxRotVelocity>
-        <motorType>velocity</motorType>
-        <rotorVelocitySlowdownSim>1</rotorVelocitySlowdownSim>
+        <!-- <rotorVelocitySlowdownSim>100</rotorVelocitySlowdownSim> -->
+      </plugin>
+      <!-- Motor 2: bidirectional tail thruster (signed force) -->
+      <plugin filename="gz-sim-thruster-system"
+              name="gz::sim::systems::Thruster">
+        <!-- Use the same namespace and joint as before -->
+        <namespace>${namespace}</namespace>
+        <joint_name>bot_rud_part1_bot_rud_motor_joint</joint_name>
+        <min_thrust_cmd>-1000</min_thrust_cmd>
+        <max_thrust_cmd>1000</max_thrust_cmd>
+        <!-- <deadband>0.1</deadband> -->
+        <!-- Apply force directly (not velocity control) -->
+        <velocity_control>false</velocity_control>
+        <propeller_diameter>0.08</propeller_diameter>
+        <thrust_coefficient>1.0</thrust_coefficient>
       </plugin>
     </gazebo>
